File: fpga/hw-r2/profile-drive/profile-drive.kicad_sch (KiCad schematic)
At the start: 0 parts

Commit message: more fixes, and r2 gerber first pass
Other:
- note added: "Global nets: the power rails, JTAG_* (both ends on the Configuration sheet) and FPGA_REBOOT (FPGA power sheet to Configuration). Everything else stays inside its sheet."
- note removed: "Global nets: the power rails, USB_DP/USB_DM (Power to UART sheet) and JTAG_* (Configuration to UART sheet). Everything else stays inside its sheet."
Changed lines of the file:
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@@
   (text "microSD socket in SPI mode" (exclude_from_sim no) (at 109.22 154.94 0) (effects (font (size 1.27 1.27)) (justify left top)))
   (text "console header, status LEDs" (exclude_from_sim no) (at 203.2 154.94 0) (effects (font (size 1.27 1.27)) (justify left top)))
-  (text "Global nets: the power rails, USB_DP/USB_DM (Power to UART sheet) and JTAG_* (Configuration to UART sheet).\nEverything else stays inside its sheet." (exclude_from_sim no) (at 15.24 177.8 0) (effects (font (size 1.27 1.27)) (justify left top)))
+  (text "Global nets: the power rails, JTAG_* (both ends on the Configuration sheet) and FPGA_REBOOT (FPGA power sheet to Configuration).\nEverything else stays inside its sheet." (exclude_from_sim no) (at 15.24 177.8 0) (effects (font (size 1.27 1.27)) (justify left top)))
   (sheet (at 15.24 43.18) (size 81.28 38.1) (fields_autoplaced yes) (stroke (width 0.1524) (type solid)) (fill (color 0 0 0 0.0))
     (property "Sheetname" "Power" (at 15.24 42.48 0) (effects (font (size 1.27 1.27)) (justify left bottom)))
