File: fpga/hw-r2/profile-drive/fpga_power.kicad_sch (KiCad schematic)
At the start: 25 parts, among them U1 LFE5U-12F-6TG144C

Commit message: more fixes, and r2 gerber first pass
Parts:
- C11, C12, C13, C14, C15, C16, C20, C21, C22, C23, C24, C25, C26, C27, C28, C29, C30, C31, C32: MPN (none) -> Samsung CL10B104KO8NNNC
- C17, C18, C19, C33, C34: MPN (none) -> Murata GRM188R61E106MA73D
- U1: MPN (none) -> Lattice LFE5U-12F-6TG144C
Connections:
- net FPGA_REBOOT: now reaches U1.67 (IO)
- no-connect marks 61 -> 60
Other:
- note added: "+1V1: 100n x6 at VCC pins 20, 29, 38, 66, 83, 130; 10u x3 (C17 to C19) at the 1V1 buck's output"
- note added: "+3V3: 100n x9 at VCCIO pins 9, 16, 36, 43, 70, 86, 100, 122, 137; 10u x2 (C33, C34) on the 3V3 buck's side"
- note removed: "+1V1: 100n x6 at VCC pins 20, 29, 38, 66, 83, 130; 10u x3 near the package"
- note removed: "+3V3: 100n x9 at VCCIO pins 9, 16, 36, 43, 70, 86, 100, 122, 137; 10u x2 near the package"

Commit message: finally passing; added case too
Parts:
- removed C17: 10u, Capacitor_SMD:C_0603_1608Metric, symbol device:C
- added R53: 2k2, Resistor_SMD:R_0603_1608Metric, symbol device:R
Connections:
- net +3V3: now also R53.1
- net U3_OE_N: now reaches U1.76 (IO)
- net U3_OE_N: now also R53.2
- no-connect marks 60 -> 59
Other:
- note added: "R53: U3 stays off (OE high) until the gateware drives U3_OE_N low."
Changed lines of the file:
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@@
     (title "FPGA power")
     (date "2026-09-03")
-    (rev "0.3")
+    (rev "r2")
   )
   (text "FPGA supply pins with their decoupling: one 100 nF per supply pin placed at the pin, one 10 uF per rail near the package (TN-02038 3.1). VCCAUX comes from VCCAUX_F, the ferrite-filtered 2.5 V." (exclude_from_sim no) (at 15.24 15.24 0) (effects (font (size 1.5 1.5)) (justify left top)))
@@
     (instances (project "profile-drive" (path "/a55e218f-75e5-4ac7-a1a1-30827bd7ace5/e2f17ad7-9b02-5741-ab72-64abac11d991" (reference "C16") (unit 1))))
   )
-  (symbol (lib_id "device:C") (at 105.41 100.33 0) (unit 1)
-    (exclude_from_sim no) (in_bom yes) (on_board yes) (dnp no)
-    (property "Reference" "C17" (at 108.2 99.06 0) (effects (font (size 1.27 1.27)) (justify left)))
-    (property "Value" "10u" (at 108.2 101.6 0) (effects (font (size 1.27 1.27)) (justify left)))
-    (property "Footprint" "Capacitor_SMD:C_0603_1608Metric" (at 105.41 100.33 0) (effects (font (size 1.27 1.27)) hide))
-    (property "Datasheet" "" (at 105.41 100.33 0) (effects (font (size 1.27 1.27)) hide))
-    (property "Description" "capacitor" (at 105.41 100.33 0) (effects (font (size 1.27 1.27)) hide))
-    (property "MPN" "Murata GRM188R61E106MA73D" (at 105.41 100.33 0) (effects (font (size 1.27 1.27)) hide))
-    (pin "1")
-    (pin "2")
-    (instances (project "profile-drive" (path "/a55e218f-75e5-4ac7-a1a1-30827bd7ace5/e2f17ad7-9b02-5741-ab72-64abac11d991" (reference "C17") (unit 1))))
-  )
   (symbol (lib_id "device:C") (at 95.25 100.33 0) (unit 1)
     (exclude_from_sim no) (in_bom yes) (on_board yes) (dnp no)
@@
   (junction (at 125.73 97.79) (diameter 0) (color 0 0 0 0))
   (junction (at 115.57 97.79) (diameter 0) (color 0 0 0 0))
-  (junction (at 105.41 97.79) (diameter 0) (color 0 0 0 0))
   (junction (at 95.25 97.79) (diameter 0) (color 0 0 0 0))
   (wire (pts (xy 166.37 102.87) (xy 156.21 102.87)) (stroke (width 0) (type default)))
@@
   (junction (at 125.73 102.87) (diameter 0) (color 0 0 0 0))
   (junction (at 115.57 102.87) (diameter 0) (color 0 0 0 0))
-  (junction (at 105.41 102.87) (diameter 0) (color 0 0 0 0))
   (junction (at 95.25 102.87) (diameter 0) (color 0 0 0 0))
   (wire (pts (xy 85.09 102.87) (xy 85.09 106.68)) (stroke (width 0) (type default)))
@@
   (no_connect (at 368.3 228.6))
   (no_connect (at 393.7 152.4))
-  (no_connect (at 393.7 154.94))
   (no_connect (at 393.7 157.48))
   (no_connect (at 393.7 160.02))
@@
     (property "Intersheetrefs" "${INTERSHEET_REFS}" (at 0 0 0) (effects (font (size 1.27 1.27)) hide))
   )
-  (sheet_instances (path "/" (page "3")))
+    (wire (pts (xy 393.7 154.94) (xy 401.32 154.94)) (stroke (width 0) (type default)))
+  (wire (pts (xy 398.78 151.13) (xy 398.78 154.94)) (stroke (width 0) (type default)))
+  (junction (at 398.78 154.94) (diameter 0) (color 0 0 0 0))
+  (global_label "U3_OE_N" (shape output) (at 401.32 154.94 0) (fields_autoplaced yes) (effects (font (size 1.27 1.27)) (justify left))
+    (property "Intersheetrefs" "${INTERSHEET_REFS}" (at 0 0 0) (effects (font (size 1.27 1.27)) hide)))
+  (symbol (lib_id "device:R") (at 398.78 147.32 0) (unit 1)
+    (exclude_from_sim no) (in_bom yes) (on_board yes) (dnp no)
+    (property "Reference" "R53" (at 401.07 146.05 0) (effects (font (size 1.27 1.27)) (justify left)))
+    (property "Value" "2k2" (at 401.07 148.59 0) (effects (font (size 1.27 1.27)) (justify left)))
+    (property "Footprint" "Resistor_SMD:R_0603_1608Metric" (at 398.78 147.32 0) (effects (font (size 1.27 1.27)) hide))
+    (property "Datasheet" "" (at 398.78 147.32 0) (effects (font (size 1.27 1.27)) hide))
+    (property "Description" "resistor" (at 398.78 147.32 0) (effects (font (size 1.27 1.27)) hide))
+    (property "MPN" "Yageo RC0603FR-072K2L" (at 398.78 147.32 0) (effects (font (size 1.27 1.27)) hide))
+    (pin "1")
+    (pin "2")
+    (instances (project "profile-drive" (path "/a55e218f-75e5-4ac7-a1a1-30827bd7ace5/e2f17ad7-9b02-5741-ab72-64abac11d991" (reference "R53") (unit 1))))
+  )
+  (symbol (lib_id "device:P3V3") (at 398.78 143.51 0) (unit 1)
+    (exclude_from_sim no) (in_bom no) (on_board yes) (dnp no)
+    (property "Reference" "#PWR914" (at 398.78 143.51 0) (effects (font (size 1.27 1.27)) hide))
+    (property "Value" "+3V3" (at 398.78 138.43 0) (effects (font (size 1.27 1.27))))
+    (property "Footprint" "" (at 398.78 143.51 0) (effects (font (size 1.27 1.27)) hide))
+    (property "Datasheet" "" (at 398.78 143.51 0) (effects (font (size 1.27 1.27)) hide))
+    (property "Description" "" (at 398.78 143.51 0) (effects (font (size 1.27 1.27)) hide))
+    (pin "1")
+    (instances (project "profile-drive" (path "/a55e218f-75e5-4ac7-a1a1-30827bd7ace5/e2f17ad7-9b02-5741-ab72-64abac11d991" (reference "#PWR914") (unit 1))))
+  )
+  (text "R53: U3 stays off (OE high) until the gateware drives U3_OE_N low." (exclude_from_sim no) (at 393.7 167.64 0) (effects (font (size 1.27 1.27)) (justify left top)))
+(sheet_instances (path "/" (page "3")))
 )

Commit message: cleaning up: adding BoM for builds, part numbers, DNP flags, etc.
Parts:
- C11, C12, C13, C14, C15, C16, C20, C21, C22, C23, C24, C25, C26, C27, C28, C29, C30, C31, C32: LCSC (none) -> C66501
- C18, C19, C33, C34: LCSC (none) -> C91606
- R53: LCSC (none) -> C114662
- U1: LCSC (none) -> C19979181
Changed lines of the file:
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@@
     (property "Description" "ECP5, built as a 25F" (at 203.2 127 0) (effects (font (size 1.27 1.27)) hide))
     (property "MPN" "Lattice LFE5U-12F-6TG144C" (at 203.2 127 0) (effects (font (size 1.27 1.27)) hide))
+    (property "LCSC" "C19979181" (at 203.2 127 0) (effects (font (size 1.27 1.27)) hide))
     (pin "20")
     (pin "29")
@@
     (property "Description" "capacitor" (at 166.37 100.33 0) (effects (font (size 1.27 1.27)) hide))
     (property "MPN" "Samsung CL10B104KO8NNNC" (at 166.37 100.33 0) (effects (font (size 1.27 1.27)) hide))
+    (property "LCSC" "C66501" (at 166.37 100.33 0) (effects (font (size 1.27 1.27)) hide))
     (pin "1")
     (pin "2")
@@
     (property "Description" "capacitor" (at 156.21 100.33 0) (effects (font (size 1.27 1.27)) hide))
     (property "MPN" "Samsung CL10B104KO8NNNC" (at 156.21 100.33 0) (effects (font (size 1.27 1.27)) hide))
+    (property "LCSC" "C66501" (at 156.21 100.33 0) (effects (font (size 1.27 1.27)) hide))
     (pin "1")
     (pin "2")
@@
     (property "Description" "capacitor" (at 146.05 100.33 0) (effects (font (size 1.27 1.27)) hide))
     (property "MPN" "Samsung CL10B104KO8NNNC" (at 146.05 100.33 0) (effects (font (size 1.27 1.27)) hide))
+    (property "LCSC" "C66501" (at 146.05 100.33 0) (effects (font (size 1.27 1.27)) hide))
     (pin "1")
     (pin "2")
@@
     (property "Description" "capacitor" (at 135.89 100.33 0) (effects (font (size 1.27 1.27)) hide))
     (property "MPN" "Samsung CL10B104KO8NNNC" (at 135.89 100.33 0) (effects (font (size 1.27 1.27)) hide))
+    (property "LCSC" "C66501" (at 135.89 100.33 0) (effects (font (size 1.27 1.27)) hide))
     (pin "1")
     (pin "2")
@@
     (property "Description" "capacitor" (at 125.73 100.33 0) (effects (font (size 1.27 1.27)) hide))
     (property "MPN" "Samsung CL10B104KO8NNNC" (at 125.73 100.33 0) (effects (font (size 1.27 1.27)) hide))
+    (property "LCSC" "C66501" (at 125.73 100.33 0) (effects (font (size 1.27 1.27)) hide))
     (pin "1")
     (pin "2")
@@
     (property "Description" "capacitor" (at 115.57 100.33 0) (effects (font (size 1.27 1.27)) hide))
     (property "MPN" "Samsung CL10B104KO8NNNC" (at 115.57 100.33 0) (effects (font (size 1.27 1.27)) hide))
+    (property "LCSC" "C66501" (at 115.57 100.33 0) (effects (font (size 1.27 1.27)) hide))
     (pin "1")
     (pin "2")
@@
     (property "Description" "capacitor" (at 95.25 100.33 0) (effects (font (size 1.27 1.27)) hide))
     (property "MPN" "Murata GRM188R61E106MA73D" (at 95.25 100.33 0) (effects (font (size 1.27 1.27)) hide))
+    (property "LCSC" "C91606" (at 95.25 100.33 0) (effects (font (size 1.27 1.27)) hide))
     (pin "1")
     (pin "2")
@@
     (property "Description" "capacitor" (at 85.09 100.33 0) (effects (font (size 1.27 1.27)) hide))
     (property "MPN" "Murata GRM188R61E106MA73D" (at 85.09 100.33 0) (effects (font (size 1.27 1.27)) hide))
+    (property "LCSC" "C91606" (at 85.09 100.33 0) (effects (font (size 1.27 1.27)) hide))
     (pin "1")
     (pin "2")
@@
     (property "Description" "capacitor" (at 156.21 125.73 0) (effects (font (size 1.27 1.27)) hide))
     (property "MPN" "Samsung CL10B104KO8NNNC" (at 156.21 125.73 0) (effects (font (size 1.27 1.27)) hide))
+    (property "LCSC" "C66501" (at 156.21 125.73 0) (effects (font (size 1.27 1.27)) hide))
     (pin "1")
     (pin "2")
@@
     (property "Description" "capacitor" (at 146.05 125.73 0) (effects (font (size 1.27 1.27)) hide))
     (property "MPN" "Samsung CL10B104KO8NNNC" (at 146.05 125.73 0) (effects (font (size 1.27 1.27)) hide))
+    (property "LCSC" "C66501" (at 146.05 125.73 0) (effects (font (size 1.27 1.27)) hide))
     (pin "1")
     (pin "2")
@@
     (property "Description" "capacitor" (at 135.89 125.73 0) (effects (font (size 1.27 1.27)) hide))
     (property "MPN" "Samsung CL10B104KO8NNNC" (at 135.89 125.73 0) (effects (font (size 1.27 1.27)) hide))
+    (property "LCSC" "C66501" (at 135.89 125.73 0) (effects (font (size 1.27 1.27)) hide))
     (pin "1")
     (pin "2")
@@
     (property "Description" "capacitor" (at 125.73 125.73 0) (effects (font (size 1.27 1.27)) hide))
     (property "MPN" "Samsung CL10B104KO8NNNC" (at 125.73 125.73 0) (effects (font (size 1.27 1.27)) hide))
+    (property "LCSC" "C66501" (at 125.73 125.73 0) (effects (font (size 1.27 1.27)) hide))
     (pin "1")
     (pin "2")
@@
     (property "Description" "capacitor" (at 240.03 100.33 0) (effects (font (size 1.27 1.27)) hide))
     (property "MPN" "Samsung CL10B104KO8NNNC" (at 240.03 100.33 0) (effects (font (size 1.27 1.27)) hide))
+    (property "LCSC" "C66501" (at 240.03 100.33 0) (effects (font (size 1.27 1.27)) hide))
     (pin "1")
     (pin "2")
@@
     (property "Description" "capacitor" (at 250.19 100.33 0) (effects (font (size 1.27 1.27)) hide))
     (property "MPN" "Samsung CL10B104KO8NNNC" (at 250.19 100.33 0) (effects (font (size 1.27 1.27)) hide))
+    (property "LCSC" "C66501" (at 250.19 100.33 0) (effects (font (size 1.27 1.27)) hide))
     (pin "1")
     (pin "2")
@@
     (property "Description" "capacitor" (at 260.35 100.33 0) (effects (font (size 1.27 1.27)) hide))
     (property "MPN" "Samsung CL10B104KO8NNNC" (at 260.35 100.33 0) (effects (font (size 1.27 1.27)) hide))
+    (property "LCSC" "C66501" (at 260.35 100.33 0) (effects (font (size 1.27 1.27)) hide))
     (pin "1")
     (pin "2")
@@
     (property "Description" "capacitor" (at 270.51 100.33 0) (effects (font (size 1.27 1.27)) hide))
     (property "MPN" "Samsung CL10B104KO8NNNC" (at 270.51 100.33 0) (effects (font (size 1.27 1.27)) hide))
+    (property "LCSC" "C66501" (at 270.51 100.33 0) (effects (font (size 1.27 1.27)) hide))
     (pin "1")
     (pin "2")
@@
     (property "Description" "capacitor" (at 280.67 100.33 0) (effects (font (size 1.27 1.27)) hide))
     (property "MPN" "Samsung CL10B104KO8NNNC" (at 280.67 100.33 0) (effects (font (size 1.27 1.27)) hide))
+    (property "LCSC" "C66501" (at 280.67 100.33 0) (effects (font (size 1.27 1.27)) hide))
     (pin "1")
     (pin "2")
@@
     (property "Description" "capacitor" (at 290.83 100.33 0) (effects (font (size 1.27 1.27)) hide))
     (property "MPN" "Samsung CL10B104KO8NNNC" (at 290.83 100.33 0) (effects (font (size 1.27 1.27)) hide))
+    (property "LCSC" "C66501" (at 290.83 100.33 0) (effects (font (size 1.27 1.27)) hide))
     (pin "1")
     (pin "2")
@@
     (property "Description" "capacitor" (at 300.99 100.33 0) (effects (font (size 1.27 1.27)) hide))
     (property "MPN" "Samsung CL10B104KO8NNNC" (at 300.99 100.33 0) (effects (font (size 1.27 1.27)) hide))
+    (property "LCSC" "C66501" (at 300.99 100.33 0) (effects (font (size 1.27 1.27)) hide))
     (pin "1")
     (pin "2")
@@
     (property "Description" "capacitor" (at 311.15 100.33 0) (effects (font (size 1.27 1.27)) hide))
     (property "MPN" "Samsung CL10B104KO8NNNC" (at 311.15 100.33 0) (effects (font (size 1.27 1.27)) hide))
+    (property "LCSC" "C66501" (at 311.15 100.33 0) (effects (font (size 1.27 1.27)) hide))
     (pin "1")
     (pin "2")
@@
     (property "Description" "capacitor" (at 321.31 100.33 0) (effects (font (size 1.27 1.27)) hide))
     (property "MPN" "Samsung CL10B104KO8NNNC" (at 321.31 100.33 0) (effects (font (size 1.27 1.27)) hide))
+    (property "LCSC" "C66501" (at 321.31 100.33 0) (effects (font (size 1.27 1.27)) hide))
     (pin "1")
     (pin "2")
@@
     (property "Description" "capacitor" (at 331.47 100.33 0) (effects (font (size 1.27 1.27)) hide))
     (property "MPN" "Murata GRM188R61E106MA73D" (at 331.47 100.33 0) (effects (font (size 1.27 1.27)) hide))
+    (property "LCSC" "C91606" (at 331.47 100.33 0) (effects (font (size 1.27 1.27)) hide))
     (pin "1")
     (pin "2")
@@
     (property "Description" "capacitor" (at 341.63 100.33 0) (effects (font (size 1.27 1.27)) hide))
     (property "MPN" "Murata GRM188R61E106MA73D" (at 341.63 100.33 0) (effects (font (size 1.27 1.27)) hide))
+    (property "LCSC" "C91606" (at 341.63 100.33 0) (effects (font (size 1.27 1.27)) hide))
     (pin "1")
     (pin "2")
@@
     (property "Description" "ECP5, built as a 25F" (at 381 190.5 0) (effects (font (size 1.27 1.27)) hide))
     (property "MPN" "Lattice LFE5U-12F-6TG144C" (at 381 190.5 0) (effects (font (size 1.27 1.27)) hide))
+    (property "LCSC" "C19979181" (at 381 190.5 0) (effects (font (size 1.27 1.27)) hide))
     (pin "11")
     (pin "12")
@@
     (property "Description" "resistor" (at 398.78 147.32 0) (effects (font (size 1.27 1.27)) hide))
     (property "MPN" "Yageo RC0603FR-072K2L" (at 398.78 147.32 0) (effects (font (size 1.27 1.27)) hide))
-    (pin "1")
-    (pin "2")
+    (property "LCSC" "C114662" (at 398.78 147.32 0) (effects (font (size 1.27 1.27)) hide))
+    (pin "1")
+    (pin "2")
