File: fpga/hw-r2/profile-drive/power.kicad_sch (KiCad schematic)
At the start: 19 parts, among them J1 USB-C 16p, U5 TLV62568DBV 1V1, U6 TLV62568DBV 3V3, U7 TLV73325PDBV 2V5

Commit message: fixups, tweaking
Parts:
- added C38, C39: 10u, Capacitor_SMD:C_0603_1608Metric, symbol device:C
Connections:
- net +5V: now also C38.1, C39.1
- net GND: now also C38.2, C39.2
Other:
- note added: "1.1 V core: TLV62568, 10 uF at VIN, 2.2 uH, 22 uF; FB divider 100k / 120k"
- note added: "3.3 V IO: TLV62568, 10 uF at VIN, 2.2 uH, 22 uF; FB divider 270k / 60.4k"
- note removed: "1.1 V core: TLV62568, 2.2 uH, 22 uF; FB divider 100k / 120k"
- note removed: "3.3 V IO: TLV62568, 2.2 uH, 22 uF; FB divider 270k / 60.4k"
Changed lines of the file:
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@@
   )
   (rectangle (start 15.24 114.3) (end 190.5 175.26) (stroke (width 0.2) (type dash)) (fill (type none)))
-  (text "1.1 V core: TLV62568, 2.2 uH, 22 uF; FB divider 100k / 120k" (exclude_from_sim no) (at 16.51 111 0) (effects (font (size 2 2) bold) (justify left top)))
+  (text "1.1 V core: TLV62568, 10 uF at VIN, 2.2 uH, 22 uF; FB divider 100k / 120k" (exclude_from_sim no) (at 16.51 111 0) (effects (font (size 2 2) bold) (justify left top)))
   (symbol (lib_id "device:TLV62568") (at 63.5 139.7 0) (unit 1)
     (exclude_from_sim no) (in_bom yes) (on_board yes) (dnp no)
@@
   (label "FB_1V1" (at 77.47 140.97 0) (fields_autoplaced yes) (effects (font (size 1.27 1.27)) (justify left bottom)))
   (rectangle (start 15.24 177.8) (end 190.5 238.76) (stroke (width 0.2) (type dash)) (fill (type none)))
-  (text "3.3 V IO: TLV62568, 2.2 uH, 22 uF; FB divider 270k / 60.4k" (exclude_from_sim no) (at 16.51 174.5 0) (effects (font (size 2 2) bold) (justify left top)))
+  (text "3.3 V IO: TLV62568, 10 uF at VIN, 2.2 uH, 22 uF; FB divider 270k / 60.4k" (exclude_from_sim no) (at 16.51 174.5 0) (effects (font (size 2 2) bold) (justify left top)))
   (symbol (lib_id "device:TLV62568") (at 63.5 203.2 0) (unit 1)
     (exclude_from_sim no) (in_bom yes) (on_board yes) (dnp no)
@@
   (text "Rails" (exclude_from_sim no) (at 203.2 38.1 0) (effects (font (size 2 2) bold) (justify left top)))
   (text "+5V       USB VBUS, bucks in\n+3V3      FPGA VCCIO, flash, oscillator, SD, 74LVC245 A side, LDO in\n+1V1      FPGA core\n+2V5      LDO output, only FB1 hangs on it\nVCCAUX_F  FPGA VCCAUX, after the ferrite\nGND       one plane" (exclude_from_sim no) (at 203.2 45.72 0) (effects (font (size 1.27 1.27)) (justify left top)))
+  (symbol (lib_id "device:C") (at 40.64 140.97 0) (unit 1)
+    (exclude_from_sim no) (in_bom yes) (on_board yes) (dnp no)
+    (property "Reference" "C38" (at 42.93 139.7 0) (effects (font (size 1.27 1.27)) (justify left)))
+    (property "Value" "10u" (at 42.93 142.24 0) (effects (font (size 1.27 1.27)) (justify left)))
+    (property "Footprint" "Capacitor_SMD:C_0603_1608Metric" (at 40.64 140.97 0) (effects (font (size 1.27 1.27)) hide))
+    (property "Datasheet" "" (at 40.64 140.97 0) (effects (font (size 1.27 1.27)) hide))
+    (property "Description" "capacitor" (at 40.64 140.97 0) (effects (font (size 1.27 1.27)) hide))
+    (pin "1")
+    (pin "2")
+    (instances (project "profile-drive" (path "/a55e218f-75e5-4ac7-a1a1-30827bd7ace5/52653336-3db4-5871-a322-379b0d9ed0e5" (reference "C38") (unit 1))))
+  )
+  (wire (pts (xy 40.64 138.43) (xy 49.53 138.43)) (stroke (width 0) (type default)))
+  (junction (at 49.53 138.43) (diameter 0) (color 0 0 0 0))
+  (symbol (lib_id "device:GND") (at 40.64 143.51 0) (unit 1)
+    (exclude_from_sim no) (in_bom no) (on_board yes) (dnp no)
+    (property "Reference" "#PWR903" (at 42.93 142.24 0) (effects (font (size 1.27 1.27)) hide))
+    (property "Value" "GND" (at 42.93 144.78 0) (effects (font (size 1.27 1.27)) (justify left)))
+    (property "Footprint" "" (at 40.64 143.51 0) (effects (font (size 1.27 1.27)) hide))
+    (property "Datasheet" "" (at 40.64 143.51 0) (effects (font (size 1.27 1.27)) hide))
+    (property "Description" "" (at 40.64 143.51 0) (effects (font (size 1.27 1.27)) hide))
+    (pin "1")
+    (instances (project "profile-drive" (path "/a55e218f-75e5-4ac7-a1a1-30827bd7ace5/52653336-3db4-5871-a322-379b0d9ed0e5" (reference "#PWR903") (unit 1))))
+  )
+  (symbol (lib_id "device:C") (at 40.64 204.47 0) (unit 1)
+    (exclude_from_sim no) (in_bom yes) (on_board yes) (dnp no)
+    (property "Reference" "C39" (at 42.93 203.2 0) (effects (font (size 1.27 1.27)) (justify left)))
+    (property "Value" "10u" (at 42.93 205.74 0) (effects (font (size 1.27 1.27)) (justify left)))
+    (property "Footprint" "Capacitor_SMD:C_0603_1608Metric" (at 40.64 204.47 0) (effects (font (size 1.27 1.27)) hide))
+    (property "Datasheet" "" (at 40.64 204.47 0) (effects (font (size 1.27 1.27)) hide))
+    (property "Description" "capacitor" (at 40.64 204.47 0) (effects (font (size 1.27 1.27)) hide))
+    (pin "1")
+    (pin "2")
+    (instances (project "profile-drive" (path "/a55e218f-75e5-4ac7-a1a1-30827bd7ace5/52653336-3db4-5871-a322-379b0d9ed0e5" (reference "C39") (unit 1))))
+  )
+  (wire (pts (xy 40.64 201.93) (xy 49.53 201.93)) (stroke (width 0) (type default)))
+  (junction (at 49.53 201.93) (diameter 0) (color 0 0 0 0))
+  (symbol (lib_id "device:GND") (at 40.64 207.01 0) (unit 1)
+    (exclude_from_sim no) (in_bom no) (on_board yes) (dnp no)
+    (property "Reference" "#PWR904" (at 42.93 205.74 0) (effects (font (size 1.27 1.27)) hide))
+    (property "Value" "GND" (at 42.93 208.28 0) (effects (font (size 1.27 1.27)) (justify left)))
+    (property "Footprint" "" (at 40.64 207.01 0) (effects (font (size 1.27 1.27)) hide))
+    (property "Datasheet" "" (at 40.64 207.01 0) (effects (font (size 1.27 1.27)) hide))
+    (property "Description" "" (at 40.64 207.01 0) (effects (font (size 1.27 1.27)) hide))
+    (pin "1")
+    (instances (project "profile-drive" (path "/a55e218f-75e5-4ac7-a1a1-30827bd7ace5/52653336-3db4-5871-a322-379b0d9ed0e5" (reference "#PWR904") (unit 1))))
+  )
   (sheet_instances (path "/" (page "2")))
 )

Commit message: more fixes, and r2 gerber first pass
Parts:
- C1, C38, C39, C9: MPN (none) -> Murata GRM188R61E106MA73D
- C10: MPN (none) -> Samsung CL10B105KA8NNNC
- C2, C3, C4: MPN (none) -> Samsung CL31A226KAHNNNE
- FB1: MPN (none) -> Murata BLM18PG121SN1D
- J1: MPN (none) -> GCT USB4105-GF-A
- L1, L2: value 2u2 -> 1u0; footprint Inductor_SMD_Wurth:L_Wurth_WE-LQSH-4020 -> device:L_Murata_DFE252012F; MPN (none) -> Murata DFE252012F-1R0M=P2
- R29, R30: MPN (none) -> Yageo RC0603FR-075K1L
- R31: value 100k -> 84.5k; MPN (none) -> Yageo RC0603FR-0784K5L
- R32: value 120k -> 100k; MPN (none) -> Yageo RC0603FR-07100KL
- R33: MPN (none) -> Yageo RC0603FR-07270KL
- R34: MPN (none) -> Yageo RC0603FR-0760K4L
- U5: value TLV62568DBV 1V1 -> TPS62A01A 1V1; footprint Package_TO_SOT_SMD:SOT-23-5_HandSoldering -> Package_TO_SOT_SMD:SOT-23-6_Handsoldering; symbol device:TLV62568 -> device:TPS62A01A; MPN (none) -> TI TPS62A01APDDCR
- U6: value TLV62568DBV 3V3 -> TPS62A01A 3V3; footprint Package_TO_SOT_SMD:SOT-23-5_HandSoldering -> Package_TO_SOT_SMD:SOT-23-6_Handsoldering; symbol device:TLV62568 -> device:TPS62A01A; MPN (none) -> TI TPS62A01APDDCR
- U7: MPN (none) -> TI TLV73325PDBVR
Connections:
- net FB_1V1: now also U5.6 (FB); no longer U5.5 (FB)
- net FB_3V3: now also U6.6 (FB); no longer U6.5 (FB)
- no-connect marks 3 -> 5
Other:
- note added: "1.1 V core: TPS62A01A (forced PWM, 2.4 MHz), 10 uF at VIN, 1.0 uH, 22 uF; FB divider 84.5k / 100k"
- note added: "3.3 V IO: TPS62A01A (forced PWM, 2.4 MHz), 10 uF at VIN, 1.0 uH, 22 uF; FB divider 270k / 60.4k"
- note added: "Power: a single USB-C cable supplies 5 V. Two TPS62A01A forced-PWM bucks make 1.1 V (core) and 3.3 V (IO); a TLV733 LDO makes 2.5 V for VCCAUX, filtered through FB1."
- note added: "USB-C input, CC sink declaration"
- note removed: "1.1 V core: TLV62568, 10 uF at VIN, 2.2 uH, 22 uF; FB divider 100k / 120k"
- note removed: "3.3 V IO: TLV62568, 10 uF at VIN, 2.2 uH, 22 uF; FB divider 270k / 60.4k"
- note removed: "Power: a single USB-C cable supplies 5 V. Two TLV62568 bucks make 1.1 V (core) and 3.3 V (IO); a TLV733 LDO makes 2.5 V for VCCAUX, filtered through FB1."
- note removed: "USB-C input, CC sink declaration, ESD"

Commit message: finally passing; added case too
Parts:
- added C40: 100u, Capacitor_SMD:CP_Elec_6.3x5.8, symbol device:C_Polarized
- added D9: SMF5.0A, Diode_SMD:D_SOD-123F, symbol device:D_Zener
- J1: footprint Connector_USB:USB_C_Receptacle_GCT_USB4105-xx-A_16P_TopMnt_Horizontal -> device:USB_C_Receptacle_GCT_USB4105-xx-A_16P_TopMnt_Horizontal
- R33: value 270k -> 274k; MPN Yageo RC0603FR-07270KL -> Yageo RC0603FR-07274KL
Connections:
- net +5V: now also C40.1, D9.1 (K)
- net GND: now also C40.2, D9.2 (A)
Other:
- note added: "3.3 V IO: TPS62A01A (forced PWM, 2.4 MHz), 10 uF at VIN, 1.0 uH, 22 uF; FB divider 274k / 60.4k (3.322 V)"
- note added: "A live USB-A to C cable hot-plugged into the all-ceramic input rings toward twice VBUS (LT AN88). C40 (100u electrolytic, about 0.36 ohm ESR) damps the ring. D9 (SMF5.0A, 6.4 V min breakdown) limits what is left. D9 alone cannot hold the bucks' 6.5 V limit."
- note removed: "3.3 V IO: TPS62A01A (forced PWM, 2.4 MHz), 10 uF at VIN, 1.0 uH, 22 uF; FB divider 270k / 60.4k"
Changed lines of the file:
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@@
     (title "Power")
     (date "2026-09-03")
-    (rev "0.3")
+    (rev "r2")
   )
   (text "Power: a single USB-C cable supplies 5 V. Two TPS62A01A forced-PWM bucks make 1.1 V (core) and 3.3 V (IO); a TLV733 LDO makes 2.5 V for VCCAUX, filtered through FB1." (exclude_from_sim no) (at 15.24 15.24 0) (effects (font (size 1.5 1.5)) (justify left top)))
@@
     (property "Reference" "J1" (at 30.48 40 0) (effects (font (size 1.27 1.27)) (justify left)))
     (property "Value" "USB-C 16p" (at 30.48 42.55 0) (effects (font (size 1.27 1.27)) (justify left)))
-    (property "Footprint" "Connector_USB:USB_C_Receptacle_GCT_USB4105-xx-A_16P_TopMnt_Horizontal" (at 38.1 63.5 0) (effects (font (size 1.27 1.27)) hide))
+    (property "Footprint" "device:USB_C_Receptacle_GCT_USB4105-xx-A_16P_TopMnt_Horizontal" (at 38.1 63.5 0) (effects (font (size 1.27 1.27)) hide))
     (property "Datasheet" "" (at 38.1 63.5 0) (effects (font (size 1.27 1.27)) hide))
     (property "Description" "USB-C receptacle, USB 2.0; A/B pads stacked" (at 38.1 63.5 0) (effects (font (size 1.27 1.27)) hide))
@@
   (label "FB_1V1" (at 77.47 140.97 0) (fields_autoplaced yes) (effects (font (size 1.27 1.27)) (justify left bottom)))
   (rectangle (start 15.24 177.8) (end 190.5 238.76) (stroke (width 0.2) (type dash)) (fill (type none)))
-  (text "3.3 V IO: TPS62A01A (forced PWM, 2.4 MHz), 10 uF at VIN, 1.0 uH, 22 uF; FB divider 270k / 60.4k" (exclude_from_sim no) (at 16.51 174.5 0) (effects (font (size 2 2) bold) (justify left top)))
+  (text "3.3 V IO: TPS62A01A (forced PWM, 2.4 MHz), 10 uF at VIN, 1.0 uH, 22 uF; FB divider 274k / 60.4k (3.322 V)" (exclude_from_sim no) (at 16.51 174.5 0) (effects (font (size 2 2) bold) (justify left top)))
   (symbol (lib_id "device:TPS62A01A") (at 63.5 203.2 0) (unit 1)
     (exclude_from_sim no) (in_bom yes) (on_board yes) (dnp no)
@@
     (exclude_from_sim no) (in_bom yes) (on_board yes) (dnp no)
     (property "Reference" "R33" (at 126.75 204.47 0) (effects (font (size 1.27 1.27)) (justify left)))
-    (property "Value" "270k" (at 126.75 207.01 0) (effects (font (size 1.27 1.27)) (justify left)))
+    (property "Value" "274k" (at 126.75 207.01 0) (effects (font (size 1.27 1.27)) (justify left)))
     (property "Footprint" "Resistor_SMD:R_0603_1608Metric" (at 124.46 205.74 0) (effects (font (size 1.27 1.27)) hide))
     (property "Datasheet" "" (at 124.46 205.74 0) (effects (font (size 1.27 1.27)) hide))
     (property "Description" "resistor" (at 124.46 205.74 0) (effects (font (size 1.27 1.27)) hide))
-    (property "MPN" "Yageo RC0603FR-07270KL" (at 124.46 205.74 0) (effects (font (size 1.27 1.27)) hide))
+    (property "MPN" "Yageo RC0603FR-07274KL" (at 124.46 205.74 0) (effects (font (size 1.27 1.27)) hide))
     (pin "1")
     (pin "2")
@@
   (no_connect (at 63.5 130.81))
   (no_connect (at 63.5 194.31))
-  (sheet_instances (path "/" (page "2")))
+    (symbol (lib_id "device:D_Zener") (at 76.2 46.99 270) (unit 1)
+    (exclude_from_sim no) (in_bom yes) (on_board yes) (dnp no)
+    (property "Reference" "D9" (at 78.74 45.72 0) (effects (font (size 1.27 1.27)) (justify left)))
+    (property "Value" "SMF5.0A" (at 78.74 48.26 0) (effects (font (size 1.27 1.27)) (justify left)))
+    (property "Footprint" "Diode_SMD:D_SOD-123F" (at 76.2 46.99 0) (effects (font (size 1.27 1.27)) hide))
+    (property "Datasheet" "" (at 76.2 46.99 0) (effects (font (size 1.27 1.27)) hide))
+    (property "Description" "5 V unidirectional TVS on VBUS" (at 76.2 46.99 0) (effects (font (size 1.27 1.27)) hide))
+    (property "MPN" "Littelfuse SMF5.0A" (at 76.2 46.99 0) (effects (font (size 1.27 1.27)) hide))
+    (pin "1")
+    (pin "2")
+    (instances (project "profile-drive" (path "/a55e218f-75e5-4ac7-a1a1-30827bd7ace5/52653336-3db4-5871-a322-379b0d9ed0e5" (reference "D9") (unit 1))))
+  )
+  (symbol (lib_id "device:GND") (at 76.2 50.8 0) (unit 1)
+    (exclude_from_sim no) (in_bom no) (on_board yes) (dnp no)
+    (property "Reference" "#PWR913" (at 76.2 50.8 0) (effects (font (size 1.27 1.27)) hide))
+    (property "Value" "GND" (at 76.2 55.24 0) (effects (font (size 1.27 1.27))))
+    (property "Footprint" "" (at 76.2 50.8 0) (effects (font (size 1.27 1.27)) hide))
+    (property "Datasheet" "" (at 76.2 50.8 0) (effects (font (size 1.27 1.27)) hide))
+    (property "Description" "" (at 76.2 50.8 0) (effects (font (size 1.27 1.27)) hide))
+    (pin "1")
+    (instances (project "profile-drive" (path "/a55e218f-75e5-4ac7-a1a1-30827bd7ace5/52653336-3db4-5871-a322-379b0d9ed0e5" (reference "#PWR913") (unit 1))))
+  )
+  (wire (pts (xy 66.04 43.18) (xy 76.2 43.18)) (stroke (width 0) (type default)))
+  (junction (at 66.04 43.18) (diameter 0) (color 0 0 0 0))
+  (text "A live USB-A to C cable hot-plugged into the all-ceramic input rings toward twice VBUS (LT AN88). C40 (100u electrolytic, about\n0.36 ohm ESR) damps the ring. D9 (SMF5.0A, 6.4 V min breakdown) limits what is left. D9 alone cannot hold the bucks' 6.5 V limit." (exclude_from_sim no) (at 17.78 100.33 0) (effects (font (size 1.27 1.27)) (justify left top)))
+  (symbol (lib_id "device:C_Polarized") (at 86.36 46.99 0) (unit 1)
+    (exclude_from_sim no) (in_bom yes) (on_board yes) (dnp no)
+    (property "Reference" "C40" (at 88.9 45.72 0) (effects (font (size 1.27 1.27)) (justify left)))
+    (property "Value" "100u" (at 88.9 48.26 0) (effects (font (size 1.27 1.27)) (justify left)))
+    (property "Footprint" "Capacitor_SMD:CP_Elec_6.3x5.8" (at 86.36 46.99 0) (effects (font (size 1.27 1.27)) hide))
+    (property "Datasheet" "" (at 86.36 46.99 0) (effects (font (size 1.27 1.27)) hide))
+    (property "Description" "16 V aluminum electrolytic, about 0.36 ohm ESR: damps the cable ringing on VBUS" (at 86.36 46.99 0) (effects (font (size 1.27 1.27)) hide))
+    (property "MPN" "Panasonic EEE-FK1C101P" (at 86.36 46.99 0) (effects (font (size 1.27 1.27)) hide))
+    (pin "1")
+    (pin "2")
+    (instances (project "profile-drive" (path "/a55e218f-75e5-4ac7-a1a1-30827bd7ace5/52653336-3db4-5871-a322-379b0d9ed0e5" (reference "C40") (unit 1))))
+  )
+  (symbol (lib_id "device:GND") (at 86.36 50.8 0) (unit 1)
+    (exclude_from_sim no) (in_bom no) (on_board yes) (dnp no)
+    (property "Reference" "#PWR915" (at 86.36 50.8 0) (effects (font (size 1.27 1.27)) hide))
+    (property "Value" "GND" (at 86.36 55.24 0) (effects (font (size 1.27 1.27))))
+    (property "Footprint" "" (at 86.36 50.8 0) (effects (font (size 1.27 1.27)) hide))
+    (property "Datasheet" "" (at 86.36 50.8 0) (effects (font (size 1.27 1.27)) hide))
+    (property "Description" "" (at 86.36 50.8 0) (effects (font (size 1.27 1.27)) hide))
+    (pin "1")
+    (instances (project "profile-drive" (path "/a55e218f-75e5-4ac7-a1a1-30827bd7ace5/52653336-3db4-5871-a322-379b0d9ed0e5" (reference "#PWR915") (unit 1))))
+  )
+  (wire (pts (xy 76.2 43.18) (xy 86.36 43.18)) (stroke (width 0) (type default)))
+  (junction (at 76.2 43.18) (diameter 0) (color 0 0 0 0))
+(sheet_instances (path "/" (page "2")))
 )
