File: fpga/hw-r2/profile-drive/power.kicad_sch (KiCad schematic)
At the start: 23 parts, among them J1 USB-C 16p, U5 TPS62A01A 1V1, U6 TPS62A01A 3V3, U7 TLV73325PDBV 2V5

Commit message: cleaning up: adding BoM for builds, part numbers, DNP flags, etc.
Parts:
- C1, C38, C39, C9: LCSC (none) -> C91606
- C10: LCSC (none) -> C29936
- C2, C3, C4: LCSC (none) -> C12891
- C40: LCSC (none) -> C128532
- D9: LCSC (none) -> C151296
- FB1: LCSC (none) -> C14709
- J1: LCSC (none) -> C3020560
- L1, L2: LCSC (none) -> C435392
- R29, R30: LCSC (none) -> C105580
- R31: LCSC (none) -> C326920
- R32: LCSC (none) -> C14675
- R33: LCSC (none) -> C482818
- R34: LCSC (none) -> C165742
- U5, U6: LCSC (none) -> C41730179
- U7: LCSC (none) -> C882825
Changed lines of the file:
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@@
     (property "Description" "USB-C receptacle, USB 2.0; A/B pads stacked" (at 38.1 63.5 0) (effects (font (size 1.27 1.27)) hide))
     (property "MPN" "GCT USB4105-GF-A" (at 38.1 63.5 0) (effects (font (size 1.27 1.27)) hide))
+    (property "LCSC" "C3020560" (at 38.1 63.5 0) (effects (font (size 1.27 1.27)) hide))
     (pin "A4")
     (pin "A6")
@@
     (property "Description" "capacitor" (at 66.04 45.72 0) (effects (font (size 1.27 1.27)) hide))
     (property "MPN" "Samsung CL31A226KAHNNNE" (at 66.04 45.72 0) (effects (font (size 1.27 1.27)) hide))
+    (property "LCSC" "C12891" (at 66.04 45.72 0) (effects (font (size 1.27 1.27)) hide))
     (pin "1")
     (pin "2")
@@
     (property "Description" "resistor" (at 58.42 63.5 0) (effects (font (size 1.27 1.27)) hide))
     (property "MPN" "Yageo RC0603FR-075K1L" (at 58.42 63.5 0) (effects (font (size 1.27 1.27)) hide))
+    (property "LCSC" "C105580" (at 58.42 63.5 0) (effects (font (size 1.27 1.27)) hide))
     (pin "1")
     (pin "2")
@@
     (property "Description" "resistor" (at 58.42 68.58 0) (effects (font (size 1.27 1.27)) hide))
     (property "MPN" "Yageo RC0603FR-075K1L" (at 58.42 68.58 0) (effects (font (size 1.27 1.27)) hide))
+    (property "LCSC" "C105580" (at 58.42 68.58 0) (effects (font (size 1.27 1.27)) hide))
     (pin "1")
     (pin "2")
@@
     (property "Description" "1 A synchronous buck, forced PWM" (at 63.5 139.7 0) (effects (font (size 1.27 1.27)) hide))
     (property "MPN" "TI TPS62A01APDDCR" (at 63.5 139.7 0) (effects (font (size 1.27 1.27)) hide))
+    (property "LCSC" "C41730179" (at 63.5 139.7 0) (effects (font (size 1.27 1.27)) hide))
     (pin "6")
     (pin "4")
@@
     (property "Description" "inductor" (at 90.17 138.43 0) (effects (font (size 1.27 1.27)) hide))
     (property "MPN" "Murata DFE252012F-1R0M=P2" (at 90.17 138.43 0) (effects (font (size 1.27 1.27)) hide))
+    (property "LCSC" "C435392" (at 90.17 138.43 0) (effects (font (size 1.27 1.27)) hide))
     (pin "1")
     (pin "2")
@@
     (property "Description" "capacitor" (at 106.68 140.97 0) (effects (font (size 1.27 1.27)) hide))
     (property "MPN" "Samsung CL31A226KAHNNNE" (at 106.68 140.97 0) (effects (font (size 1.27 1.27)) hide))
+    (property "LCSC" "C12891" (at 106.68 140.97 0) (effects (font (size 1.27 1.27)) hide))
     (pin "1")
     (pin "2")
@@
     (property "Description" "resistor" (at 124.46 142.24 0) (effects (font (size 1.27 1.27)) hide))
     (property "MPN" "Yageo RC0603FR-0784K5L" (at 124.46 142.24 0) (effects (font (size 1.27 1.27)) hide))
+    (property "LCSC" "C326920" (at 124.46 142.24 0) (effects (font (size 1.27 1.27)) hide))
     (pin "1")
     (pin "2")
@@
     (property "Description" "resistor" (at 124.46 149.86 0) (effects (font (size 1.27 1.27)) hide))
     (property "MPN" "Yageo RC0603FR-07100KL" (at 124.46 149.86 0) (effects (font (size 1.27 1.27)) hide))
+    (property "LCSC" "C14675" (at 124.46 149.86 0) (effects (font (size 1.27 1.27)) hide))
     (pin "1")
     (pin "2")
@@
     (property "Description" "1 A synchronous buck, forced PWM" (at 63.5 203.2 0) (effects (font (size 1.27 1.27)) hide))
     (property "MPN" "TI TPS62A01APDDCR" (at 63.5 203.2 0) (effects (font (size 1.27 1.27)) hide))
+    (property "LCSC" "C41730179" (at 63.5 203.2 0) (effects (font (size 1.27 1.27)) hide))
     (pin "6")
     (pin "4")
@@
     (property "Description" "inductor" (at 90.17 201.93 0) (effects (font (size 1.27 1.27)) hide))
     (property "MPN" "Murata DFE252012F-1R0M=P2" (at 90.17 201.93 0) (effects (font (size 1.27 1.27)) hide))
+    (property "LCSC" "C435392" (at 90.17 201.93 0) (effects (font (size 1.27 1.27)) hide))
     (pin "1")
     (pin "2")
@@
     (property "Description" "capacitor" (at 106.68 204.47 0) (effects (font (size 1.27 1.27)) hide))
     (property "MPN" "Samsung CL31A226KAHNNNE" (at 106.68 204.47 0) (effects (font (size 1.27 1.27)) hide))
+    (property "LCSC" "C12891" (at 106.68 204.47 0) (effects (font (size 1.27 1.27)) hide))
     (pin "1")
     (pin "2")
@@
     (property "Description" "resistor" (at 124.46 205.74 0) (effects (font (size 1.27 1.27)) hide))
     (property "MPN" "Yageo RC0603FR-07274KL" (at 124.46 205.74 0) (effects (font (size 1.27 1.27)) hide))
+    (property "LCSC" "C482818" (at 124.46 205.74 0) (effects (font (size 1.27 1.27)) hide))
     (pin "1")
     (pin "2")
@@
     (property "Description" "resistor" (at 124.46 213.36 0) (effects (font (size 1.27 1.27)) hide))
     (property "MPN" "Yageo RC0603FR-0760K4L" (at 124.46 213.36 0) (effects (font (size 1.27 1.27)) hide))
+    (property "LCSC" "C165742" (at 124.46 213.36 0) (effects (font (size 1.27 1.27)) hide))
     (pin "1")
     (pin "2")
@@
     (property "Description" "300 mA LDO" (at 63.5 266.7 0) (effects (font (size 1.27 1.27)) hide))
     (property "MPN" "TI TLV73325PDBVR" (at 63.5 266.7 0) (effects (font (size 1.27 1.27)) hide))
+    (property "LCSC" "C882825" (at 63.5 266.7 0) (effects (font (size 1.27 1.27)) hide))
     (pin "1")
     (pin "3")
@@
     (property "Description" "capacitor" (at 41.91 267.97 0) (effects (font (size 1.27 1.27)) hide))
     (property "MPN" "Samsung CL10B105KA8NNNC" (at 41.91 267.97 0) (effects (font (size 1.27 1.27)) hide))
+    (property "LCSC" "C29936" (at 41.91 267.97 0) (effects (font (size 1.27 1.27)) hide))
     (pin "1")
     (pin "2")
@@
     (property "Description" "capacitor" (at 77.47 267.97 0) (effects (font (size 1.27 1.27)) hide))
     (property "MPN" "Murata GRM188R61E106MA73D" (at 77.47 267.97 0) (effects (font (size 1.27 1.27)) hide))
+    (property "LCSC" "C91606" (at 77.47 267.97 0) (effects (font (size 1.27 1.27)) hide))
     (pin "1")
     (pin "2")
@@
     (property "Description" "ferrite bead" (at 95.25 265.43 0) (effects (font (size 1.27 1.27)) hide))
     (property "MPN" "Murata BLM18PG121SN1D" (at 95.25 265.43 0) (effects (font (size 1.27 1.27)) hide))
+    (property "LCSC" "C14709" (at 95.25 265.43 0) (effects (font (size 1.27 1.27)) hide))
     (pin "1")
     (pin "2")
@@
     (property "Description" "capacitor" (at 121.92 267.97 0) (effects (font (size 1.27 1.27)) hide))
     (property "MPN" "Murata GRM188R61E106MA73D" (at 121.92 267.97 0) (effects (font (size 1.27 1.27)) hide))
+    (property "LCSC" "C91606" (at 121.92 267.97 0) (effects (font (size 1.27 1.27)) hide))
     (pin "1")
     (pin "2")
@@
     (property "Description" "capacitor" (at 40.64 140.97 0) (effects (font (size 1.27 1.27)) hide))
     (property "MPN" "Murata GRM188R61E106MA73D" (at 40.64 140.97 0) (effects (font (size 1.27 1.27)) hide))
+    (property "LCSC" "C91606" (at 40.64 140.97 0) (effects (font (size 1.27 1.27)) hide))
     (pin "1")
     (pin "2")
@@
     (property "Description" "capacitor" (at 40.64 204.47 0) (effects (font (size 1.27 1.27)) hide))
     (property "MPN" "Murata GRM188R61E106MA73D" (at 40.64 204.47 0) (effects (font (size 1.27 1.27)) hide))
+    (property "LCSC" "C91606" (at 40.64 204.47 0) (effects (font (size 1.27 1.27)) hide))
     (pin "1")
     (pin "2")
@@
     (property "Description" "5 V unidirectional TVS on VBUS" (at 76.2 46.99 0) (effects (font (size 1.27 1.27)) hide))
     (property "MPN" "Littelfuse SMF5.0A" (at 76.2 46.99 0) (effects (font (size 1.27 1.27)) hide))
+    (property "LCSC" "C151296" (at 76.2 46.99 0) (effects (font (size 1.27 1.27)) hide))
     (pin "1")
     (pin "2")
@@
     (property "Description" "16 V aluminum electrolytic, about 0.36 ohm ESR: damps the cable ringing on VBUS" (at 86.36 46.99 0) (effects (font (size 1.27 1.27)) hide))
     (property "MPN" "Panasonic EEE-FK1C101P" (at 86.36 46.99 0) (effects (font (size 1.27 1.27)) hide))
-    (pin "1")
-    (pin "2")
+    (property "LCSC" "C128532" (at 86.36 46.99 0) (effects (font (size 1.27 1.27)) hide))
+    (pin "1")
+    (pin "2")
