File: fpga/hw-r2/profile-drive/profile_bus.kicad_sch (KiCad schematic)
At the start: 13 parts, among them J2 DB-25F right-angle, U1 LFE5U-12F-6TG144C, U2 74LVC245A DATA, U3 74LVC245A CTRL-IN

Commit message: fixups, tweaking
Parts:
- J2: value DB-25F right-angle -> NorComp 182-025-213R561; footprint Connector_Dsub:DSUB-25_Socket_Horizontal_P2.77x2.84mm_EdgePinOffset4.94mm_Housed_MountingHolesOffset4.94mm -> device:DSUB-25_Female_Horizontal_NorComp_182-025-213R561
Changed lines of the file:
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@@
     (exclude_from_sim no) (in_bom yes) (on_board yes) (dnp no)
     (property "Reference" "J2" (at 359.41 85.72 0) (effects (font (size 1.27 1.27)) (justify left)))
-    (property "Value" "DB-25F right-angle" (at 359.41 88.27 0) (effects (font (size 1.27 1.27)) (justify left)))
-    (property "Footprint" "Connector_Dsub:DSUB-25_Socket_Horizontal_P2.77x2.84mm_EdgePinOffset4.94mm_Housed_MountingHolesOffset4.94mm" (at 368.3 114.3 0) (effects (font (size 1.27 1.27)) hide))
+    (property "Value" "NorComp 182-025-213R561" (at 359.41 88.27 0) (effects (font (size 1.27 1.27)) (justify left)))
+    (property "Footprint" "device:DSUB-25_Female_Horizontal_NorComp_182-025-213R561" (at 368.3 114.3 0) (effects (font (size 1.27 1.27)) hide))
     (property "Datasheet" "" (at 368.3 114.3 0) (effects (font (size 1.27 1.27)) hide))
     (property "Description" "ProFile port, DB-25 female" (at 368.3 114.3 0) (effects (font (size 1.27 1.27)) hide))

Commit message: more fixes, and r2 gerber first pass
Parts:
- added RN1, RN2, RN3, RN4: 47R, Resistor_SMD:R_Array_Convex_4x0603, symbol device:R_Pack04
- C35, C36: MPN (none) -> Samsung CL10B104KO8NNNC
- J2: MPN (none) -> NorComp 182-025-213R561
- R1, R2, R3: MPN (none) -> Yageo RC0603FR-07220RL
- R14, R15: MPN (none) -> Yageo RC0603FR-07100KL
- R4, R5: MPN (none) -> Yageo RC0603FR-0710KL
- U1: MPN (none) -> Lattice LFE5U-12F-6TG144C
- U2, U3: MPN (none) -> TI SN74LVC245APWR
Connections:
- net at U1.102 (FPGA_PRES_N): now also RN3.4; no longer U3.5 (A4)
- net at U1.103 (FPGA_PH0): now also RN4.1; no longer U3.6 (A5)
- net at U1.104 (FPGA_AUX7): now also RN4.2; no longer U3.7 (A6)
- net at U1.88 (FPGA_PD0): now also RN1.1; no longer U2.2 (A1)
- net at U1.89 (FPGA_PD1): now also RN1.2; no longer U2.3 (A2)
- net at U1.90 (FPGA_PD2): now also RN1.3; no longer U2.4 (A3)
- net at U1.91 (FPGA_PD3): now also RN1.4; no longer U2.5 (A4)
- net at U1.92 (FPGA_PD4): now also RN2.1; no longer U2.6 (A5)
- net at U1.93 (FPGA_PD5): now also RN2.2; no longer U2.7 (A6)
- net at U1.94 (FPGA_PD6): now also RN2.3; no longer U2.8 (A7)
- net at U1.95 (FPGA_PD7): now also RN2.4; no longer U2.9 (A8)
- net at U1.97 (FPGA_PCMD_N): now also RN3.1; no longer U3.2 (A1)
- net at U1.98 (FPGA_PSTRB_N): now also RN3.2; no longer U3.3 (A2)
- net at U1.99 (FPGA_PRW): now also RN3.3; no longer U3.4 (A3)
- new net: RN1.5, U2.5 (A4)
- new net: RN1.6, U2.4 (A3)
- new net: RN1.7, U2.3 (A2)
- new net: RN1.8, U2.2 (A1)
- new net: RN3.8, U3.2 (A1)
- new net: RN3.7, U3.3 (A2)
- new net: RN3.6, U3.4 (A3)
- new net: RN3.5, U3.5 (A4)
- new net: RN4.8, U3.6 (A5)
- new net: RN4.7, U3.7 (A6)
- new net: RN2.8, U2.6 (A5)
- new net: RN2.7, U2.7 (A6)
- new net: RN2.6, U2.8 (A7)
- new net: RN2.5, U2.9 (A8)
- no-connect marks 2 -> 6
Other:
- note added: "J2 pin numbers are the ProFile cable's; the drive is the socket end. R14/R15 keep PH0 and AUX7 low with no cable attached."
- note added: "RN1 to RN4: 47R in series at the 74LVC245A A outputs, for source termination. Simulated 2026-10-09: without them the fast corner rings back into the threshold band on the long strobe lines."
- note removed: "J2 pin numbers are the ProFile cable's; the drive is the socket end. R15/R15 keep PH0 and AUX7 low with no cable attached."

Commit message: finally passing; added case too
Parts:
- removed R15: 100k, Resistor_SMD:R_0603_1608Metric, symbol device:R
- added R49, R50, R51, R52: 100k, Resistor_SMD:R_0603_1608Metric, symbol device:R
- R14: value 100k -> 47k; MPN Yageo RC0603FR-07100KL -> Yageo RC0603FR-0747KL
- R4: value 10k -> 2k2; MPN Yageo RC0603FR-0710KL -> Yageo RC0603FR-072K2L
- R5: value 10k -> 100k; MPN Yageo RC0603FR-0710KL -> Yageo RC0603FR-07100KL
- RN1, RN2, RN3, RN4: footprint Resistor_SMD:R_Array_Convex_4x0603 -> device:R_Array_Convex_4x0603_Yageo_YC164
Connections:
- net +3V3: now also U3.13 (B6), R49.1, R50.1, R51.1, R52.1; no longer U3.19 (/OE)
- net PCMD_N: now also R49.2
- net PRES_N: now also R52.2
- net PRW: now also R51.2
- net PSTRB_N: now also R50.2
- net at U1.104 (FPGA_AUX7): no longer RN4.2
- net at U3.7 (A6): no longer RN4.7
- net AUX7: no longer names the net of J2.7 (AUX7)
- net AUX7: no longer U3.13 (B6)
- new net U3_OE_N: U3.19 (/OE)
- no-connect marks 6 -> 11
Other:
- note added: "J2 pin numbers are the ProFile cable's; the drive is the socket end. R14 keeps PH0 low with no cable attached. Pin 7 is N/C on the ProFile and the //e card, so it is not used: U3 B6 is grounded and U1 pin 104 (the C/D partner of PRES_N's pin 102) is open."
- note added: "ProFile bus. U2 carries the eight data lines both ways (DIR and /OE from the FPGA). U3 brings the five host-driven control lines in (pin 7, AUX7, is N/C and unused). /PBSY, /PPARITY and PCHK are driven by the FPGA through 220 R. All ProFile-side nets are 5 V."
- note added: "R49 to R52: U3's host-side inputs (PCMD_N, PSTRB_N, PRW, PRES_N) idle high with no cable or the host off. TI requires a 74LVC245A's inputs held at a rail (PH0 has R14 to GND; B6 to B8 are grounded)."
- note added: "U3 is held off (OE high, R53) until the gateware drives U3_OE_N low after configuration: U1 pins 97/99 are an ECP5 A/B pair. The pair must not be driven apart before the core supply passes POR (Lattice FPGA-DS-02012 3.6). The host can hold them apart."
- note added: "U3: B to A only (DIR = 0); /OE on U3_OE_N (R53 holds it off until the gateware drives U1 pin 76 low); unused B6 to B8 grounded."
- note removed: "J2 pin numbers are the ProFile cable's; the drive is the socket end. R14/R15 keep PH0 and AUX7 low with no cable attached."
- note removed: "ProFile bus. U2 carries the eight data lines both ways (DIR and /OE from the FPGA). U3 brings the six host-driven control lines in. /PBSY, /PPARITY and PCHK are driven by the FPGA through 220 R. All ProFile-side nets are 5 V."
- note removed: "U3: B to A only (DIR = 0, /OE = 0); unused B7/B8 grounded."

Commit message: cleaning up: adding BoM for builds, part numbers, DNP flags, etc.
Parts:
- C35, C36: LCSC (none) -> C66501
- J2: LCSC (none) -> C17257261
- R1, R2, R3: LCSC (none) -> C107696
- R14: LCSC (none) -> C105579
- R4: LCSC (none) -> C114662
- R49, R5, R50, R51, R52: LCSC (none) -> C14675
- RN1, RN2, RN3, RN4: LCSC (none) -> C606217
- U1: LCSC (none) -> C19979181
- U2, U3: LCSC (none) -> C7848
Changed lines of the file:
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@@
     (property "Description" "ECP5, built as a 25F" (at 50.8 152.4 0) (effects (font (size 1.27 1.27)) hide))
     (property "MPN" "Lattice LFE5U-12F-6TG144C" (at 50.8 152.4 0) (effects (font (size 1.27 1.27)) hide))
+    (property "LCSC" "C19979181" (at 50.8 152.4 0) (effects (font (size 1.27 1.27)) hide))
     (pin "73")
     (pin "74")
@@
     (property "Description" "octal bus transceiver, 3.3 V side A, 5 V tolerant" (at 114.3 118.11 0) (effects (font (size 1.27 1.27)) hide))
     (property "MPN" "TI SN74LVC245APWR" (at 114.3 118.11 0) (effects (font (size 1.27 1.27)) hide))
+    (property "LCSC" "C7848" (at 114.3 118.11 0) (effects (font (size 1.27 1.27)) hide))
     (pin "1")
     (pin "19")
@@
     (property "Description" "resistor" (at 71.12 102.87 0) (effects (font (size 1.27 1.27)) hide))
     (property "MPN" "Yageo RC0603FR-07100KL" (at 71.12 102.87 0) (effects (font (size 1.27 1.27)) hide))
+    (property "LCSC" "C14675" (at 71.12 102.87 0) (effects (font (size 1.27 1.27)) hide))
     (pin "1")
     (pin "2")
@@
     (property "Description" "resistor" (at 83.82 100.33 0) (effects (font (size 1.27 1.27)) hide))
     (property "MPN" "Yageo RC0603FR-072K2L" (at 83.82 100.33 0) (effects (font (size 1.27 1.27)) hide))
+    (property "LCSC" "C114662" (at 83.82 100.33 0) (effects (font (size 1.27 1.27)) hide))
     (pin "1")
     (pin "2")
@@
     (property "Description" "capacitor" (at 132.08 97.79 0) (effects (font (size 1.27 1.27)) hide))
     (property "MPN" "Samsung CL10B104KO8NNNC" (at 132.08 97.79 0) (effects (font (size 1.27 1.27)) hide))
+    (property "LCSC" "C66501" (at 132.08 97.79 0) (effects (font (size 1.27 1.27)) hide))
     (pin "1")
     (pin "2")
@@
     (property "Description" "octal bus transceiver, 3.3 V side A, 5 V tolerant" (at 114.3 168.91 0) (effects (font (size 1.27 1.27)) hide))
     (property "MPN" "TI SN74LVC245APWR" (at 114.3 168.91 0) (effects (font (size 1.27 1.27)) hide))
+    (property "LCSC" "C7848" (at 114.3 168.91 0) (effects (font (size 1.27 1.27)) hide))
     (pin "1")
     (pin "19")
@@
     (property "Description" "capacitor" (at 132.08 148.59 0) (effects (font (size 1.27 1.27)) hide))
     (property "MPN" "Samsung CL10B104KO8NNNC" (at 132.08 148.59 0) (effects (font (size 1.27 1.27)) hide))
+    (property "LCSC" "C66501" (at 132.08 148.59 0) (effects (font (size 1.27 1.27)) hide))
     (pin "1")
     (pin "2")
@@
     (property "Description" "resistor" (at 76.2 182.88 0) (effects (font (size 1.27 1.27)) hide))
     (property "MPN" "Yageo RC0603FR-07220RL" (at 76.2 182.88 0) (effects (font (size 1.27 1.27)) hide))
+    (property "LCSC" "C107696" (at 76.2 182.88 0) (effects (font (size 1.27 1.27)) hide))
     (pin "1")
     (pin "2")
@@
     (property "Description" "resistor" (at 76.2 190.5 0) (effects (font (size 1.27 1.27)) hide))
     (property "MPN" "Yageo RC0603FR-07220RL" (at 76.2 190.5 0) (effects (font (size 1.27 1.27)) hide))
+    (property "LCSC" "C107696" (at 76.2 190.5 0) (effects (font (size 1.27 1.27)) hide))
     (pin "1")
     (pin "2")
@@
     (property "Description" "resistor" (at 76.2 198.12 0) (effects (font (size 1.27 1.27)) hide))
     (property "MPN" "Yageo RC0603FR-07220RL" (at 76.2 198.12 0) (effects (font (size 1.27 1.27)) hide))
+    (property "LCSC" "C107696" (at 76.2 198.12 0) (effects (font (size 1.27 1.27)) hide))
     (pin "1")
     (pin "2")
@@
     (property "Description" "ProFile port, DB-25 female" (at 368.3 114.3 0) (effects (font (size 1.27 1.27)) hide))
     (property "MPN" "NorComp 182-025-213R561" (at 368.3 114.3 0) (effects (font (size 1.27 1.27)) hide))
+    (property "LCSC" "C17257261" (at 368.3 114.3 0) (effects (font (size 1.27 1.27)) hide))
     (pin "1")
     (pin "7")
@@
     (property "Description" "resistor" (at 339.09 85.09 0) (effects (font (size 1.27 1.27)) hide))
     (property "MPN" "Yageo RC0603FR-0747KL" (at 339.09 85.09 0) (effects (font (size 1.27 1.27)) hide))
+    (property "LCSC" "C105579" (at 339.09 85.09 0) (effects (font (size 1.27 1.27)) hide))
     (pin "1")
     (pin "2")
@@
     (property "Description" "47R x4 series, source termination of the 74LVC245A A outputs" (at 91.44 115.57 0) (effects (font (size 1.27 1.27)) hide))
     (property "MPN" "Yageo YC164-FR-0747RL" (at 91.44 115.57 0) (effects (font (size 1.27 1.27)) hide))
+    (property "LCSC" "C606217" (at 91.44 115.57 0) (effects (font (size 1.27 1.27)) hide))
     (pin "1")
     (pin "2")
@@
     (property "Description" "47R x4 series, source termination of the 74LVC245A A outputs" (at 91.44 125.73 0) (effects (font (size 1.27 1.27)) hide))
     (property "MPN" "Yageo YC164-FR-0747RL" (at 91.44 125.73 0) (effects (font (size 1.27 1.27)) hide))
+    (property "LCSC" "C606217" (at 91.44 125.73 0) (effects (font (size 1.27 1.27)) hide))
     (pin "1")
     (pin "2")
@@
     (property "Description" "47R x4 series, source termination of the 74LVC245A A outputs" (at 91.44 166.37 0) (effects (font (size 1.27 1.27)) hide))
     (property "MPN" "Yageo YC164-FR-0747RL" (at 91.44 166.37 0) (effects (font (size 1.27 1.27)) hide))
+    (property "LCSC" "C606217" (at 91.44 166.37 0) (effects (font (size 1.27 1.27)) hide))
     (pin "1")
     (pin "2")
@@
     (property "Description" "47R x4 series, source termination of the 74LVC245A A outputs" (at 91.44 176.53 0) (effects (font (size 1.27 1.27)) hide))
     (property "MPN" "Yageo YC164-FR-0747RL" (at 91.44 176.53 0) (effects (font (size 1.27 1.27)) hide))
+    (property "LCSC" "C606217" (at 91.44 176.53 0) (effects (font (size 1.27 1.27)) hide))
     (pin "1")
     (pin "2")
@@
     (property "Description" "resistor" (at 289.56 55.88 0) (effects (font (size 1.27 1.27)) hide))
     (property "MPN" "Yageo RC0603FR-07100KL" (at 289.56 55.88 0) (effects (font (size 1.27 1.27)) hide))
+    (property "LCSC" "C14675" (at 289.56 55.88 0) (effects (font (size 1.27 1.27)) hide))
     (pin "1")
     (pin "2")
@@
     (property "Description" "resistor" (at 299.72 55.88 0) (effects (font (size 1.27 1.27)) hide))
     (property "MPN" "Yageo RC0603FR-07100KL" (at 299.72 55.88 0) (effects (font (size 1.27 1.27)) hide))
+    (property "LCSC" "C14675" (at 299.72 55.88 0) (effects (font (size 1.27 1.27)) hide))
     (pin "1")
     (pin "2")
@@
     (property "Description" "resistor" (at 309.88 55.88 0) (effects (font (size 1.27 1.27)) hide))
     (property "MPN" "Yageo RC0603FR-07100KL" (at 309.88 55.88 0) (effects (font (size 1.27 1.27)) hide))
+    (property "LCSC" "C14675" (at 309.88 55.88 0) (effects (font (size 1.27 1.27)) hide))
     (pin "1")
     (pin "2")
@@
     (property "Description" "resistor" (at 320.04 55.88 0) (effects (font (size 1.27 1.27)) hide))
     (property "MPN" "Yageo RC0603FR-07100KL" (at 320.04 55.88 0) (effects (font (size 1.27 1.27)) hide))
-    (pin "1")
-    (pin "2")
+    (property "LCSC" "C14675" (at 320.04 55.88 0) (effects (font (size 1.27 1.27)) hide))
+    (pin "1")
+    (pin "2")
