File: fpga/hw-r2/profile-drive/sdcard.kicad_sch (KiCad schematic)
At the start: 12 parts, among them J3 microSD MEM2075, U1 LFE5U-12F-6TG144C

Commit message: fixups, tweaking
Parts:
- added R46, R47: 10k, Resistor_SMD:R_0603_1608Metric, symbol device:R
Connections:
- net +3V3: now also R46.1, R47.1
- net SD_DAT2: now reaches J3.1 (DAT2)
- net SD_DAT2: now also R47.2
- net SD_DAT1: now reaches J3.8 (DAT1)
- net SD_DAT1: now also R46.2
- no-connect marks 2 -> 0
Changed lines of the file:
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@@
     (instances (project "profile-drive" (path "/a55e218f-75e5-4ac7-a1a1-30827bd7ace5/25b76539-fb21-5813-a9db-0623d2cc98f2" (reference "#PWR016") (unit 1))))
   )
-  (no_connect (at 231.14 118.11))
-  (no_connect (at 231.14 120.65))
-  (wire (pts (xy 241.3 74.93) (xy 241.3 59.69)) (stroke (width 0) (type default)))
+      (wire (pts (xy 241.3 74.93) (xy 241.3 59.69)) (stroke (width 0) (type default)))
   (junction (at 241.3 59.69) (diameter 0) (color 0 0 0 0))
   (wire (pts (xy 241.3 59.69) (xy 241.3 52.07)) (stroke (width 0) (type default)))
@@
   )
   (text "SD_CD_N: the socket's switch closes to ground with a card inserted." (exclude_from_sim no) (at 129.54 157.48 0) (effects (font (size 1.27 1.27)) (justify left top)))
+  (wire (pts (xy 231.14 118.11) (xy 223.52 118.11)) (stroke (width 0) (type default)))
+  (label "SD_DAT1" (at 223.52 118.11 180) (fields_autoplaced yes) (effects (font (size 1.27 1.27)) (justify right bottom)))
+  (wire (pts (xy 231.14 120.65) (xy 215.9 120.65)) (stroke (width 0) (type default)))
+  (label "SD_DAT2" (at 215.9 120.65 180) (fields_autoplaced yes) (effects (font (size 1.27 1.27)) (justify right bottom)))
+  (symbol (lib_id "device:R") (at 198.12 129.54 0) (unit 1)
+    (exclude_from_sim no) (in_bom yes) (on_board yes) (dnp no)
+    (property "Reference" "R46" (at 200.41 128.27 0) (effects (font (size 1.27 1.27)) (justify left)))
+    (property "Value" "10k" (at 200.41 130.81 0) (effects (font (size 1.27 1.27)) (justify left)))
+    (property "Footprint" "Resistor_SMD:R_0603_1608Metric" (at 198.12 129.54 0) (effects (font (size 1.27 1.27)) hide))
+    (property "Datasheet" "" (at 198.12 129.54 0) (effects (font (size 1.27 1.27)) hide))
+    (property "Description" "resistor" (at 198.12 129.54 0) (effects (font (size 1.27 1.27)) hide))
+    (pin "1")
+    (pin "2")
+    (instances (project "profile-drive" (path "/a55e218f-75e5-4ac7-a1a1-30827bd7ace5/25b76539-fb21-5813-a9db-0623d2cc98f2" (reference "R46") (unit 1))))
+  )
+  (symbol (lib_id "device:P3V3") (at 198.12 125.73 0) (unit 1)
+    (exclude_from_sim no) (in_bom no) (on_board yes) (dnp no)
+    (property "Reference" "#PWR907" (at 200.41 124.46 0) (effects (font (size 1.27 1.27)) hide))
+    (property "Value" "+3V3" (at 200.41 127 0) (effects (font (size 1.27 1.27)) (justify left)))
+    (property "Footprint" "" (at 198.12 125.73 0) (effects (font (size 1.27 1.27)) hide))
+    (property "Datasheet" "" (at 198.12 125.73 0) (effects (font (size 1.27 1.27)) hide))
+    (property "Description" "" (at 198.12 125.73 0) (effects (font (size 1.27 1.27)) hide))
+    (pin "1")
+    (instances (project "profile-drive" (path "/a55e218f-75e5-4ac7-a1a1-30827bd7ace5/25b76539-fb21-5813-a9db-0623d2cc98f2" (reference "#PWR907") (unit 1))))
+  )
+  (label "SD_DAT1" (at 198.12 133.35 270) (fields_autoplaced yes) (effects (font (size 1.27 1.27)) (justify right bottom)))
+  (symbol (lib_id "device:R") (at 205.74 129.54 0) (unit 1)
+    (exclude_from_sim no) (in_bom yes) (on_board yes) (dnp no)
+    (property "Reference" "R47" (at 208.03 128.27 0) (effects (font (size 1.27 1.27)) (justify left)))
+    (property "Value" "10k" (at 208.03 130.81 0) (effects (font (size 1.27 1.27)) (justify left)))
+    (property "Footprint" "Resistor_SMD:R_0603_1608Metric" (at 205.74 129.54 0) (effects (font (size 1.27 1.27)) hide))
+    (property "Datasheet" "" (at 205.74 129.54 0) (effects (font (size 1.27 1.27)) hide))
+    (property "Description" "resistor" (at 205.74 129.54 0) (effects (font (size 1.27 1.27)) hide))
+    (pin "1")
+    (pin "2")
+    (instances (project "profile-drive" (path "/a55e218f-75e5-4ac7-a1a1-30827bd7ace5/25b76539-fb21-5813-a9db-0623d2cc98f2" (reference "R47") (unit 1))))
+  )
+  (symbol (lib_id "device:P3V3") (at 205.74 125.73 0) (unit 1)
+    (exclude_from_sim no) (in_bom no) (on_board yes) (dnp no)
+    (property "Reference" "#PWR908" (at 208.03 124.46 0) (effects (font (size 1.27 1.27)) hide))
+    (property "Value" "+3V3" (at 208.03 127 0) (effects (font (size 1.27 1.27)) (justify left)))
+    (property "Footprint" "" (at 205.74 125.73 0) (effects (font (size 1.27 1.27)) hide))
+    (property "Datasheet" "" (at 205.74 125.73 0) (effects (font (size 1.27 1.27)) hide))
+    (property "Description" "" (at 205.74 125.73 0) (effects (font (size 1.27 1.27)) hide))
+    (pin "1")
+    (instances (project "profile-drive" (path "/a55e218f-75e5-4ac7-a1a1-30827bd7ace5/25b76539-fb21-5813-a9db-0623d2cc98f2" (reference "#PWR908") (unit 1))))
+  )
+  (label "SD_DAT2" (at 205.74 133.35 270) (fields_autoplaced yes) (effects (font (size 1.27 1.27)) (justify right bottom)))
   (sheet_instances (path "/" (page "6")))
 )

Commit message: more fixes, and r2 gerber first pass
Parts:
- C7: MPN (none) -> Murata GRM188R61E106MA73D
- C8: MPN (none) -> Samsung CL10B104KO8NNNC
- J3: MPN (none) -> GCT MEM2075-00-140-01-A
- R10, R11, R12, R9: MPN (none) -> Yageo RC0603FR-0733RL
- R13, R46, R47, R6, R7, R8: MPN (none) -> Yageo RC0603FR-0710KL
- U1: MPN (none) -> Lattice LFE5U-12F-6TG144C
Changed lines of the file:
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@@
     (property "Datasheet" "" (at 45.72 96.52 0) (effects (font (size 1.27 1.27)) hide))
     (property "Description" "ECP5, built as a 25F" (at 45.72 96.52 0) (effects (font (size 1.27 1.27)) hide))
+    (property "MPN" "Lattice LFE5U-12F-6TG144C" (at 45.72 96.52 0) (effects (font (size 1.27 1.27)) hide))
     (pin "110")
     (pin "111")
@@
     (property "Datasheet" "" (at 71.12 81.28 0) (effects (font (size 1.27 1.27)) hide))
     (property "Description" "resistor" (at 71.12 81.28 0) (effects (font (size 1.27 1.27)) hide))
+    (property "MPN" "Yageo RC0603FR-0733RL" (at 71.12 81.28 0) (effects (font (size 1.27 1.27)) hide))
     (pin "1")
     (pin "2")
@@
     (property "Datasheet" "" (at 71.12 88.9 0) (effects (font (size 1.27 1.27)) hide))
     (property "Description" "resistor" (at 71.12 88.9 0) (effects (font (size 1.27 1.27)) hide))
+    (property "MPN" "Yageo RC0603FR-0733RL" (at 71.12 88.9 0) (effects (font (size 1.27 1.27)) hide))
     (pin "1")
     (pin "2")
@@
     (property "Datasheet" "" (at 71.12 96.52 0) (effects (font (size 1.27 1.27)) hide))
     (property "Description" "resistor" (at 71.12 96.52 0) (effects (font (size 1.27 1.27)) hide))
+    (property "MPN" "Yageo RC0603FR-0733RL" (at 71.12 96.52 0) (effects (font (size 1.27 1.27)) hide))
     (pin "1")
     (pin "2")
@@
     (property "Datasheet" "" (at 71.12 104.14 0) (effects (font (size 1.27 1.27)) hide))
     (property "Description" "resistor" (at 71.12 104.14 0) (effects (font (size 1.27 1.27)) hide))
+    (property "MPN" "Yageo RC0603FR-0733RL" (at 71.12 104.14 0) (effects (font (size 1.27 1.27)) hide))
     (pin "1")
     (pin "2")
@@
     (property "Datasheet" "" (at 241.3 101.6 0) (effects (font (size 1.27 1.27)) hide))
     (property "Description" "microSD push-push socket, SPI mode" (at 241.3 101.6 0) (effects (font (size 1.27 1.27)) hide))
+    (property "MPN" "GCT MEM2075-00-140-01-A" (at 241.3 101.6 0) (effects (font (size 1.27 1.27)) hide))
     (pin "2")
     (pin "3")
@@
     (property "Datasheet" "" (at 213.36 76.2 0) (effects (font (size 1.27 1.27)) hide))
     (property "Description" "resistor" (at 213.36 76.2 0) (effects (font (size 1.27 1.27)) hide))
+    (property "MPN" "Yageo RC0603FR-0710KL" (at 213.36 76.2 0) (effects (font (size 1.27 1.27)) hide))
     (pin "1")
     (pin "2")
@@
     (property "Datasheet" "" (at 205.74 76.2 0) (effects (font (size 1.27 1.27)) hide))
     (property "Description" "resistor" (at 205.74 76.2 0) (effects (font (size 1.27 1.27)) hide))
+    (property "MPN" "Yageo RC0603FR-0710KL" (at 205.74 76.2 0) (effects (font (size 1.27 1.27)) hide))
     (pin "1")
     (pin "2")
@@
     (property "Datasheet" "" (at 198.12 76.2 0) (effects (font (size 1.27 1.27)) hide))
     (property "Description" "resistor" (at 198.12 76.2 0) (effects (font (size 1.27 1.27)) hide))
+    (property "MPN" "Yageo RC0603FR-0710KL" (at 198.12 76.2 0) (effects (font (size 1.27 1.27)) hide))
     (pin "1")
     (pin "2")
@@
     (property "Datasheet" "" (at 190.5 76.2 0) (effects (font (size 1.27 1.27)) hide))
     (property "Description" "resistor" (at 190.5 76.2 0) (effects (font (size 1.27 1.27)) hide))
+    (property "MPN" "Yageo RC0603FR-0710KL" (at 190.5 76.2 0) (effects (font (size 1.27 1.27)) hide))
     (pin "1")
     (pin "2")
@@
     (property "Datasheet" "" (at 251.46 62.23 0) (effects (font (size 1.27 1.27)) hide))
     (property "Description" "capacitor" (at 251.46 62.23 0) (effects (font (size 1.27 1.27)) hide))
+    (property "MPN" "Samsung CL10B104KO8NNNC" (at 251.46 62.23 0) (effects (font (size 1.27 1.27)) hide))
     (pin "1")
     (pin "2")
@@
     (property "Datasheet" "" (at 261.62 62.23 0) (effects (font (size 1.27 1.27)) hide))
     (property "Description" "capacitor" (at 261.62 62.23 0) (effects (font (size 1.27 1.27)) hide))
+    (property "MPN" "Murata GRM188R61E106MA73D" (at 261.62 62.23 0) (effects (font (size 1.27 1.27)) hide))
     (pin "1")
     (pin "2")
@@
     (property "Datasheet" "" (at 198.12 129.54 0) (effects (font (size 1.27 1.27)) hide))
     (property "Description" "resistor" (at 198.12 129.54 0) (effects (font (size 1.27 1.27)) hide))
+    (property "MPN" "Yageo RC0603FR-0710KL" (at 198.12 129.54 0) (effects (font (size 1.27 1.27)) hide))
     (pin "1")
     (pin "2")
@@
     (property "Datasheet" "" (at 205.74 129.54 0) (effects (font (size 1.27 1.27)) hide))
     (property "Description" "resistor" (at 205.74 129.54 0) (effects (font (size 1.27 1.27)) hide))
-    (pin "1")
-    (pin "2")
+    (property "MPN" "Yageo RC0603FR-0710KL" (at 205.74 129.54 0) (effects (font (size 1.27 1.27)) hide))
+    (pin "1")
+    (pin "2")

Commit message: finally passing; added case too
Other:
- note added: "microSD in SPI mode. 33 R series on the four SPI lines at the FPGA; 10k pulls on CS, MOSI, MISO, DAT1, DAT2 (R46, R47) and card-detect at the socket."
- note removed: "microSD in SPI mode. 33 R series on the four SPI lines at the FPGA; 10k pulls on CS, MOSI, MISO and card-detect at the socket."
Changed lines of the file:
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@@
     (title "SD card")
     (date "2026-09-03")
-    (rev "0.3")
+    (rev "r2")
   )
-  (text "microSD in SPI mode. 33 R series on the four SPI lines at the FPGA; 10k pulls on CS, MOSI, MISO and card-detect at the socket." (exclude_from_sim no) (at 15.24 15.24 0) (effects (font (size 1.5 1.5)) (justify left top)))
+  (text "microSD in SPI mode. 33 R series on the four SPI lines at the FPGA; 10k pulls on CS, MOSI, MISO, DAT1, DAT2 (R46, R47) and card-detect at the socket." (exclude_from_sim no) (at 15.24 15.24 0) (effects (font (size 1.5 1.5)) (justify left top)))
   (symbol (lib_id "device:LFE5U_TQFP144") (at 45.72 96.52 0) (unit 4)
     (exclude_from_sim no) (in_bom yes) (on_board yes) (dnp no)

Commit message: cleaning up: adding BoM for builds, part numbers, DNP flags, etc.
Parts:
- C7: LCSC (none) -> C91606
- C8: LCSC (none) -> C66501
- J3: LCSC (none) -> C3029735
- R10, R11, R12, R9: LCSC (none) -> C108661
- R13, R46, R47, R6, R7, R8: LCSC (none) -> C98220
- U1: LCSC (none) -> C19979181
Changed lines of the file:
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@@
     (property "Description" "ECP5, built as a 25F" (at 45.72 96.52 0) (effects (font (size 1.27 1.27)) hide))
     (property "MPN" "Lattice LFE5U-12F-6TG144C" (at 45.72 96.52 0) (effects (font (size 1.27 1.27)) hide))
+    (property "LCSC" "C19979181" (at 45.72 96.52 0) (effects (font (size 1.27 1.27)) hide))
     (pin "110")
     (pin "111")
@@
     (property "Description" "resistor" (at 71.12 81.28 0) (effects (font (size 1.27 1.27)) hide))
     (property "MPN" "Yageo RC0603FR-0733RL" (at 71.12 81.28 0) (effects (font (size 1.27 1.27)) hide))
+    (property "LCSC" "C108661" (at 71.12 81.28 0) (effects (font (size 1.27 1.27)) hide))
     (pin "1")
     (pin "2")
@@
     (property "Description" "resistor" (at 71.12 88.9 0) (effects (font (size 1.27 1.27)) hide))
     (property "MPN" "Yageo RC0603FR-0733RL" (at 71.12 88.9 0) (effects (font (size 1.27 1.27)) hide))
+    (property "LCSC" "C108661" (at 71.12 88.9 0) (effects (font (size 1.27 1.27)) hide))
     (pin "1")
     (pin "2")
@@
     (property "Description" "resistor" (at 71.12 96.52 0) (effects (font (size 1.27 1.27)) hide))
     (property "MPN" "Yageo RC0603FR-0733RL" (at 71.12 96.52 0) (effects (font (size 1.27 1.27)) hide))
+    (property "LCSC" "C108661" (at 71.12 96.52 0) (effects (font (size 1.27 1.27)) hide))
     (pin "1")
     (pin "2")
@@
     (property "Description" "resistor" (at 71.12 104.14 0) (effects (font (size 1.27 1.27)) hide))
     (property "MPN" "Yageo RC0603FR-0733RL" (at 71.12 104.14 0) (effects (font (size 1.27 1.27)) hide))
+    (property "LCSC" "C108661" (at 71.12 104.14 0) (effects (font (size 1.27 1.27)) hide))
     (pin "1")
     (pin "2")
@@
     (property "Description" "microSD push-push socket, SPI mode" (at 241.3 101.6 0) (effects (font (size 1.27 1.27)) hide))
     (property "MPN" "GCT MEM2075-00-140-01-A" (at 241.3 101.6 0) (effects (font (size 1.27 1.27)) hide))
+    (property "LCSC" "C3029735" (at 241.3 101.6 0) (effects (font (size 1.27 1.27)) hide))
     (pin "2")
     (pin "3")
@@
     (property "Description" "resistor" (at 213.36 76.2 0) (effects (font (size 1.27 1.27)) hide))
     (property "MPN" "Yageo RC0603FR-0710KL" (at 213.36 76.2 0) (effects (font (size 1.27 1.27)) hide))
+    (property "LCSC" "C98220" (at 213.36 76.2 0) (effects (font (size 1.27 1.27)) hide))
     (pin "1")
     (pin "2")
@@
     (property "Description" "resistor" (at 205.74 76.2 0) (effects (font (size 1.27 1.27)) hide))
     (property "MPN" "Yageo RC0603FR-0710KL" (at 205.74 76.2 0) (effects (font (size 1.27 1.27)) hide))
+    (property "LCSC" "C98220" (at 205.74 76.2 0) (effects (font (size 1.27 1.27)) hide))
     (pin "1")
     (pin "2")
@@
     (property "Description" "resistor" (at 198.12 76.2 0) (effects (font (size 1.27 1.27)) hide))
     (property "MPN" "Yageo RC0603FR-0710KL" (at 198.12 76.2 0) (effects (font (size 1.27 1.27)) hide))
+    (property "LCSC" "C98220" (at 198.12 76.2 0) (effects (font (size 1.27 1.27)) hide))
     (pin "1")
     (pin "2")
@@
     (property "Description" "resistor" (at 190.5 76.2 0) (effects (font (size 1.27 1.27)) hide))
     (property "MPN" "Yageo RC0603FR-0710KL" (at 190.5 76.2 0) (effects (font (size 1.27 1.27)) hide))
+    (property "LCSC" "C98220" (at 190.5 76.2 0) (effects (font (size 1.27 1.27)) hide))
     (pin "1")
     (pin "2")
@@
     (property "Description" "capacitor" (at 251.46 62.23 0) (effects (font (size 1.27 1.27)) hide))
     (property "MPN" "Samsung CL10B104KO8NNNC" (at 251.46 62.23 0) (effects (font (size 1.27 1.27)) hide))
+    (property "LCSC" "C66501" (at 251.46 62.23 0) (effects (font (size 1.27 1.27)) hide))
     (pin "1")
     (pin "2")
@@
     (property "Description" "capacitor" (at 261.62 62.23 0) (effects (font (size 1.27 1.27)) hide))
     (property "MPN" "Murata GRM188R61E106MA73D" (at 261.62 62.23 0) (effects (font (size 1.27 1.27)) hide))
+    (property "LCSC" "C91606" (at 261.62 62.23 0) (effects (font (size 1.27 1.27)) hide))
     (pin "1")
     (pin "2")
@@
     (property "Description" "resistor" (at 198.12 129.54 0) (effects (font (size 1.27 1.27)) hide))
     (property "MPN" "Yageo RC0603FR-0710KL" (at 198.12 129.54 0) (effects (font (size 1.27 1.27)) hide))
+    (property "LCSC" "C98220" (at 198.12 129.54 0) (effects (font (size 1.27 1.27)) hide))
     (pin "1")
     (pin "2")
@@
     (property "Description" "resistor" (at 205.74 129.54 0) (effects (font (size 1.27 1.27)) hide))
     (property "MPN" "Yageo RC0603FR-0710KL" (at 205.74 129.54 0) (effects (font (size 1.27 1.27)) hide))
-    (pin "1")
-    (pin "2")
+    (property "LCSC" "C98220" (at 205.74 129.54 0) (effects (font (size 1.27 1.27)) hide))
+    (pin "1")
+    (pin "2")
