File: fpga/hw-r2/profile-drive/uart_leds.kicad_sch (KiCad schematic)
At the start: 18 parts, among them J5 console UART 1x3, U1 LFE5U-12F-6TG144C

Commit message: more fixes, and r2 gerber first pass
Parts:
- R35, R36, R37, R38, R39, R40, R41, R42: MPN (none) -> Yageo RC0603FR-071KL
- U1: MPN (none) -> Lattice LFE5U-12F-6TG144C
Changed lines of the file:
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@@
     (property "Datasheet" "" (at 50.8 73.66 0) (effects (font (size 1.27 1.27)) hide))
     (property "Description" "ECP5, built as a 25F" (at 50.8 73.66 0) (effects (font (size 1.27 1.27)) hide))
+    (property "MPN" "Lattice LFE5U-12F-6TG144C" (at 50.8 73.66 0) (effects (font (size 1.27 1.27)) hide))
     (pin "1")
     (pin "2")
@@
     (property "Datasheet" "" (at 73.66 55.88 0) (effects (font (size 1.27 1.27)) hide))
     (property "Description" "resistor" (at 73.66 55.88 0) (effects (font (size 1.27 1.27)) hide))
+    (property "MPN" "Yageo RC0603FR-071KL" (at 73.66 55.88 0) (effects (font (size 1.27 1.27)) hide))
     (pin "1")
     (pin "2")
@@
     (property "Datasheet" "" (at 73.66 60.96 0) (effects (font (size 1.27 1.27)) hide))
     (property "Description" "resistor" (at 73.66 60.96 0) (effects (font (size 1.27 1.27)) hide))
+    (property "MPN" "Yageo RC0603FR-071KL" (at 73.66 60.96 0) (effects (font (size 1.27 1.27)) hide))
     (pin "1")
     (pin "2")
@@
     (property "Datasheet" "" (at 73.66 66.04 0) (effects (font (size 1.27 1.27)) hide))
     (property "Description" "resistor" (at 73.66 66.04 0) (effects (font (size 1.27 1.27)) hide))
+    (property "MPN" "Yageo RC0603FR-071KL" (at 73.66 66.04 0) (effects (font (size 1.27 1.27)) hide))
     (pin "1")
     (pin "2")
@@
     (property "Datasheet" "" (at 73.66 71.12 0) (effects (font (size 1.27 1.27)) hide))
     (property "Description" "resistor" (at 73.66 71.12 0) (effects (font (size 1.27 1.27)) hide))
+    (property "MPN" "Yageo RC0603FR-071KL" (at 73.66 71.12 0) (effects (font (size 1.27 1.27)) hide))
     (pin "1")
     (pin "2")
@@
     (property "Datasheet" "" (at 73.66 76.2 0) (effects (font (size 1.27 1.27)) hide))
     (property "Description" "resistor" (at 73.66 76.2 0) (effects (font (size 1.27 1.27)) hide))
+    (property "MPN" "Yageo RC0603FR-071KL" (at 73.66 76.2 0) (effects (font (size 1.27 1.27)) hide))
     (pin "1")
     (pin "2")
@@
     (property "Datasheet" "" (at 73.66 81.28 0) (effects (font (size 1.27 1.27)) hide))
     (property "Description" "resistor" (at 73.66 81.28 0) (effects (font (size 1.27 1.27)) hide))
+    (property "MPN" "Yageo RC0603FR-071KL" (at 73.66 81.28 0) (effects (font (size 1.27 1.27)) hide))
     (pin "1")
     (pin "2")
@@
     (property "Datasheet" "" (at 73.66 86.36 0) (effects (font (size 1.27 1.27)) hide))
     (property "Description" "resistor" (at 73.66 86.36 0) (effects (font (size 1.27 1.27)) hide))
+    (property "MPN" "Yageo RC0603FR-071KL" (at 73.66 86.36 0) (effects (font (size 1.27 1.27)) hide))
     (pin "1")
     (pin "2")
@@
     (property "Datasheet" "" (at 73.66 91.44 0) (effects (font (size 1.27 1.27)) hide))
     (property "Description" "resistor" (at 73.66 91.44 0) (effects (font (size 1.27 1.27)) hide))
+    (property "MPN" "Yageo RC0603FR-071KL" (at 73.66 91.44 0) (effects (font (size 1.27 1.27)) hide))
     (pin "1")
     (pin "2")
@@
     (property "Datasheet" "" (at 50.8 154.94 0) (effects (font (size 1.27 1.27)) hide))
     (property "Description" "ECP5, built as a 25F" (at 50.8 154.94 0) (effects (font (size 1.27 1.27)) hide))
+    (property "MPN" "Lattice LFE5U-12F-6TG144C" (at 50.8 154.94 0) (effects (font (size 1.27 1.27)) hide))
     (pin "135")
     (pin "136")

Commit message: cleaning up: adding BoM for builds, part numbers, DNP flags, etc.
Parts:
- D1, D2, D3, D4, D5, D6, D7, D8: LCSC (none) -> C2286
- J5: now not fitted
- R35, R36, R37, R38, R39, R40, R41, R42: LCSC (none) -> C22548
- U1: LCSC (none) -> C19979181
Changed lines of the file:
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@@
     (property "Description" "ECP5, built as a 25F" (at 50.8 73.66 0) (effects (font (size 1.27 1.27)) hide))
     (property "MPN" "Lattice LFE5U-12F-6TG144C" (at 50.8 73.66 0) (effects (font (size 1.27 1.27)) hide))
+    (property "LCSC" "C19979181" (at 50.8 73.66 0) (effects (font (size 1.27 1.27)) hide))
     (pin "1")
     (pin "2")
@@
     (property "Description" "resistor" (at 73.66 55.88 0) (effects (font (size 1.27 1.27)) hide))
     (property "MPN" "Yageo RC0603FR-071KL" (at 73.66 55.88 0) (effects (font (size 1.27 1.27)) hide))
+    (property "LCSC" "C22548" (at 73.66 55.88 0) (effects (font (size 1.27 1.27)) hide))
     (pin "1")
     (pin "2")
@@
     (property "Datasheet" "" (at 86.36 55.88 0) (effects (font (size 1.27 1.27)) hide))
     (property "Description" "LED, anode pin 2, cathode pin 1" (at 86.36 55.88 0) (effects (font (size 1.27 1.27)) hide))
+    (property "LCSC" "C2286" (at 86.36 55.88 0) (effects (font (size 1.27 1.27)) hide))
     (pin "2")
     (pin "1")
@@
     (property "Description" "resistor" (at 73.66 60.96 0) (effects (font (size 1.27 1.27)) hide))
     (property "MPN" "Yageo RC0603FR-071KL" (at 73.66 60.96 0) (effects (font (size 1.27 1.27)) hide))
+    (property "LCSC" "C22548" (at 73.66 60.96 0) (effects (font (size 1.27 1.27)) hide))
     (pin "1")
     (pin "2")
@@
     (property "Datasheet" "" (at 86.36 60.96 0) (effects (font (size 1.27 1.27)) hide))
     (property "Description" "LED, anode pin 2, cathode pin 1" (at 86.36 60.96 0) (effects (font (size 1.27 1.27)) hide))
+    (property "LCSC" "C2286" (at 86.36 60.96 0) (effects (font (size 1.27 1.27)) hide))
     (pin "2")
     (pin "1")
@@
     (property "Description" "resistor" (at 73.66 66.04 0) (effects (font (size 1.27 1.27)) hide))
     (property "MPN" "Yageo RC0603FR-071KL" (at 73.66 66.04 0) (effects (font (size 1.27 1.27)) hide))
+    (property "LCSC" "C22548" (at 73.66 66.04 0) (effects (font (size 1.27 1.27)) hide))
     (pin "1")
     (pin "2")
@@
     (property "Datasheet" "" (at 86.36 66.04 0) (effects (font (size 1.27 1.27)) hide))
     (property "Description" "LED, anode pin 2, cathode pin 1" (at 86.36 66.04 0) (effects (font (size 1.27 1.27)) hide))
+    (property "LCSC" "C2286" (at 86.36 66.04 0) (effects (font (size 1.27 1.27)) hide))
     (pin "2")
     (pin "1")
@@
     (property "Description" "resistor" (at 73.66 71.12 0) (effects (font (size 1.27 1.27)) hide))
     (property "MPN" "Yageo RC0603FR-071KL" (at 73.66 71.12 0) (effects (font (size 1.27 1.27)) hide))
+    (property "LCSC" "C22548" (at 73.66 71.12 0) (effects (font (size 1.27 1.27)) hide))
     (pin "1")
     (pin "2")
@@
     (property "Datasheet" "" (at 86.36 71.12 0) (effects (font (size 1.27 1.27)) hide))
     (property "Description" "LED, anode pin 2, cathode pin 1" (at 86.36 71.12 0) (effects (font (size 1.27 1.27)) hide))
+    (property "LCSC" "C2286" (at 86.36 71.12 0) (effects (font (size 1.27 1.27)) hide))
     (pin "2")
     (pin "1")
@@
     (property "Description" "resistor" (at 73.66 76.2 0) (effects (font (size 1.27 1.27)) hide))
     (property "MPN" "Yageo RC0603FR-071KL" (at 73.66 76.2 0) (effects (font (size 1.27 1.27)) hide))
+    (property "LCSC" "C22548" (at 73.66 76.2 0) (effects (font (size 1.27 1.27)) hide))
     (pin "1")
     (pin "2")
@@
     (property "Datasheet" "" (at 86.36 76.2 0) (effects (font (size 1.27 1.27)) hide))
     (property "Description" "LED, anode pin 2, cathode pin 1" (at 86.36 76.2 0) (effects (font (size 1.27 1.27)) hide))
+    (property "LCSC" "C2286" (at 86.36 76.2 0) (effects (font (size 1.27 1.27)) hide))
     (pin "2")
     (pin "1")
@@
     (property "Description" "resistor" (at 73.66 81.28 0) (effects (font (size 1.27 1.27)) hide))
     (property "MPN" "Yageo RC0603FR-071KL" (at 73.66 81.28 0) (effects (font (size 1.27 1.27)) hide))
+    (property "LCSC" "C22548" (at 73.66 81.28 0) (effects (font (size 1.27 1.27)) hide))
     (pin "1")
     (pin "2")
@@
     (property "Datasheet" "" (at 86.36 81.28 0) (effects (font (size 1.27 1.27)) hide))
     (property "Description" "LED, anode pin 2, cathode pin 1" (at 86.36 81.28 0) (effects (font (size 1.27 1.27)) hide))
+    (property "LCSC" "C2286" (at 86.36 81.28 0) (effects (font (size 1.27 1.27)) hide))
     (pin "2")
     (pin "1")
@@
     (property "Description" "resistor" (at 73.66 86.36 0) (effects (font (size 1.27 1.27)) hide))
     (property "MPN" "Yageo RC0603FR-071KL" (at 73.66 86.36 0) (effects (font (size 1.27 1.27)) hide))
+    (property "LCSC" "C22548" (at 73.66 86.36 0) (effects (font (size 1.27 1.27)) hide))
     (pin "1")
     (pin "2")
@@
     (property "Datasheet" "" (at 86.36 86.36 0) (effects (font (size 1.27 1.27)) hide))
     (property "Description" "LED, anode pin 2, cathode pin 1" (at 86.36 86.36 0) (effects (font (size 1.27 1.27)) hide))
+    (property "LCSC" "C2286" (at 86.36 86.36 0) (effects (font (size 1.27 1.27)) hide))
     (pin "2")
     (pin "1")
@@
     (property "Description" "resistor" (at 73.66 91.44 0) (effects (font (size 1.27 1.27)) hide))
     (property "MPN" "Yageo RC0603FR-071KL" (at 73.66 91.44 0) (effects (font (size 1.27 1.27)) hide))
+    (property "LCSC" "C22548" (at 73.66 91.44 0) (effects (font (size 1.27 1.27)) hide))
     (pin "1")
     (pin "2")
@@
     (property "Datasheet" "" (at 86.36 91.44 0) (effects (font (size 1.27 1.27)) hide))
     (property "Description" "LED, anode pin 2, cathode pin 1" (at 86.36 91.44 0) (effects (font (size 1.27 1.27)) hide))
+    (property "LCSC" "C2286" (at 86.36 91.44 0) (effects (font (size 1.27 1.27)) hide))
     (pin "2")
     (pin "1")
@@
     (property "Description" "ECP5, built as a 25F" (at 50.8 154.94 0) (effects (font (size 1.27 1.27)) hide))
     (property "MPN" "Lattice LFE5U-12F-6TG144C" (at 50.8 154.94 0) (effects (font (size 1.27 1.27)) hide))
+    (property "LCSC" "C19979181" (at 50.8 154.94 0) (effects (font (size 1.27 1.27)) hide))
     (pin "135")
     (pin "136")
@@
   (label "UART_RX" (at 73.66 156.21 0) (fields_autoplaced yes) (effects (font (size 1.27 1.27)) (justify left bottom)))
   (symbol (lib_id "device:Header_UART") (at 127 154.94 0) (unit 1)
-    (exclude_from_sim no) (in_bom yes) (on_board yes) (dnp no)
+    (exclude_from_sim no) (in_bom yes) (on_board yes) (dnp yes)
     (property "Reference" "J5" (at 121.92 144.14 0) (effects (font (size 1.27 1.27)) (justify left)))
     (property "Value" "console UART 1x3" (at 121.92 146.68 0) (effects (font (size 1.27 1.27)) (justify left)))
