File: fpga/hw-r2/profile-drive/config.kicad_sch (KiCad schematic)
At the start: 23 parts, among them J4 JTAG 1x6, J6 flash service 1x7, J7 PROGRAMN button header (optio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, SW1 PROGRAMN button, U1 LFE5U-12F-6TG144C, U4 W25Q128JVSIQ, X1 25MHz XO 2520 3V3

Commit message: fixups, tweaking
Parts:
- added R43: 100R, Resistor_SMD:R_0603_1608Metric, symbol device:R
- added R44, R45: 10k, Resistor_SMD:R_0603_1608Metric, symbol device:R
Connections:
- net +3V3: now also R44.1, R45.1
- net SPI_CLK_R: now also R43.1; no longer J6.4 (CLK)
- net SPI_MISO: now also R45.2
- net SPI_MOSI: now also R44.2
- new net SPI_CLK_J6: J6.4 (CLK), R43.2
Other:
- note added: "R43 keeps the long run to J6 off the flash clock pin. R44/R45: MOSI and MISO pull-ups, TN-02039 table 4.3 note 4."
Changed lines of the file:
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@@
   (label "SPI_CS_N" (at 365.76 91.44 180) (fields_autoplaced yes) (effects (font (size 1.27 1.27)) (justify right bottom)))
   (wire (pts (xy 373.38 93.98) (xy 365.76 93.98)) (stroke (width 0) (type default)))
-  (label "SPI_CLK_R" (at 365.76 93.98 180) (fields_autoplaced yes) (effects (font (size 1.27 1.27)) (justify right bottom)))
+  (label "SPI_CLK_J6" (at 365.76 93.98 180) (fields_autoplaced yes) (effects (font (size 1.27 1.27)) (justify right bottom)))
   (wire (pts (xy 373.38 96.52) (xy 365.76 96.52)) (stroke (width 0) (type default)))
   (label "SPI_MOSI" (at 365.76 96.52 180) (fields_autoplaced yes) (effects (font (size 1.27 1.27)) (justify right bottom)))
@@
   (label "CLK25" (at 321.31 180.34 0) (fields_autoplaced yes) (effects (font (size 1.27 1.27)) (justify left bottom)))
   (text "CLK25 enters PCLKT0_0 (pin 128); the design multiplies it to 50 MHz in the PLL." (exclude_from_sim no) (at 256.54 198.12 0) (effects (font (size 1.27 1.27)) (justify left top)))
+  (symbol (lib_id "device:R") (at 347.98 93.98 90) (unit 1)
+    (exclude_from_sim no) (in_bom yes) (on_board yes) (dnp no)
+    (property "Reference" "R43" (at 350.27 92.71 0) (effects (font (size 1.27 1.27)) (justify left)))
+    (property "Value" "100R" (at 350.27 95.25 0) (effects (font (size 1.27 1.27)) (justify left)))
+    (property "Footprint" "Resistor_SMD:R_0603_1608Metric" (at 347.98 93.98 0) (effects (font (size 1.27 1.27)) hide))
+    (property "Datasheet" "" (at 347.98 93.98 0) (effects (font (size 1.27 1.27)) hide))
+    (property "Description" "resistor" (at 347.98 93.98 0) (effects (font (size 1.27 1.27)) hide))
+    (pin "1")
+    (pin "2")
+    (instances (project "profile-drive" (path "/a55e218f-75e5-4ac7-a1a1-30827bd7ace5/695229fb-70b3-528e-9b1e-e2ca33d5906b" (reference "R43") (unit 1))))
+  )
+  (label "SPI_CLK_R" (at 344.17 93.98 180) (fields_autoplaced yes) (effects (font (size 1.27 1.27)) (justify right bottom)))
+  (label "SPI_CLK_J6" (at 351.79 93.98 0) (fields_autoplaced yes) (effects (font (size 1.27 1.27)) (justify left bottom)))
+  (symbol (lib_id "device:R") (at 335.28 116.84 0) (unit 1)
+    (exclude_from_sim no) (in_bom yes) (on_board yes) (dnp no)
+    (property "Reference" "R44" (at 337.57 115.57 0) (effects (font (size 1.27 1.27)) (justify left)))
+    (property "Value" "10k" (at 337.57 118.11 0) (effects (font (size 1.27 1.27)) (justify left)))
+    (property "Footprint" "Resistor_SMD:R_0603_1608Metric" (at 335.28 116.84 0) (effects (font (size 1.27 1.27)) hide))
+    (property "Datasheet" "" (at 335.28 116.84 0) (effects (font (size 1.27 1.27)) hide))
+    (property "Description" "resistor" (at 335.28 116.84 0) (effects (font (size 1.27 1.27)) hide))
+    (pin "1")
+    (pin "2")
+    (instances (project "profile-drive" (path "/a55e218f-75e5-4ac7-a1a1-30827bd7ace5/695229fb-70b3-528e-9b1e-e2ca33d5906b" (reference "R44") (unit 1))))
+  )
+  (symbol (lib_id "device:P3V3") (at 335.28 113.03 0) (unit 1)
+    (exclude_from_sim no) (in_bom no) (on_board yes) (dnp no)
+    (property "Reference" "#PWR905" (at 337.57 111.76 0) (effects (font (size 1.27 1.27)) hide))
+    (property "Value" "+3V3" (at 337.57 114.3 0) (effects (font (size 1.27 1.27)) (justify left)))
+    (property "Footprint" "" (at 335.28 113.03 0) (effects (font (size 1.27 1.27)) hide))
+    (property "Datasheet" "" (at 335.28 113.03 0) (effects (font (size 1.27 1.27)) hide))
+    (property "Description" "" (at 335.28 113.03 0) (effects (font (size 1.27 1.27)) hide))
+    (pin "1")
+    (instances (project "profile-drive" (path "/a55e218f-75e5-4ac7-a1a1-30827bd7ace5/695229fb-70b3-528e-9b1e-e2ca33d5906b" (reference "#PWR905") (unit 1))))
+  )
+  (label "SPI_MOSI" (at 335.28 120.65 270) (fields_autoplaced yes) (effects (font (size 1.27 1.27)) (justify right bottom)))
+  (symbol (lib_id "device:R") (at 342.9 116.84 0) (unit 1)
+    (exclude_from_sim no) (in_bom yes) (on_board yes) (dnp no)
+    (property "Reference" "R45" (at 345.19 115.57 0) (effects (font (size 1.27 1.27)) (justify left)))
+    (property "Value" "10k" (at 345.19 118.11 0) (effects (font (size 1.27 1.27)) (justify left)))
+    (property "Footprint" "Resistor_SMD:R_0603_1608Metric" (at 342.9 116.84 0) (effects (font (size 1.27 1.27)) hide))
+    (property "Datasheet" "" (at 342.9 116.84 0) (effects (font (size 1.27 1.27)) hide))
+    (property "Description" "resistor" (at 342.9 116.84 0) (effects (font (size 1.27 1.27)) hide))
+    (pin "1")
+    (pin "2")
+    (instances (project "profile-drive" (path "/a55e218f-75e5-4ac7-a1a1-30827bd7ace5/695229fb-70b3-528e-9b1e-e2ca33d5906b" (reference "R45") (unit 1))))
+  )
+  (symbol (lib_id "device:P3V3") (at 342.9 113.03 0) (unit 1)
+    (exclude_from_sim no) (in_bom no) (on_board yes) (dnp no)
+    (property "Reference" "#PWR906" (at 345.19 111.76 0) (effects (font (size 1.27 1.27)) hide))
+    (property "Value" "+3V3" (at 345.19 114.3 0) (effects (font (size 1.27 1.27)) (justify left)))
+    (property "Footprint" "" (at 342.9 113.03 0) (effects (font (size 1.27 1.27)) hide))
+    (property "Datasheet" "" (at 342.9 113.03 0) (effects (font (size 1.27 1.27)) hide))
+    (property "Description" "" (at 342.9 113.03 0) (effects (font (size 1.27 1.27)) hide))
+    (pin "1")
+    (instances (project "profile-drive" (path "/a55e218f-75e5-4ac7-a1a1-30827bd7ace5/695229fb-70b3-528e-9b1e-e2ca33d5906b" (reference "#PWR906") (unit 1))))
+  )
+  (label "SPI_MISO" (at 342.9 120.65 270) (fields_autoplaced yes) (effects (font (size 1.27 1.27)) (justify right bottom)))
+  (text "R43 keeps the long run to J6 off the flash clock pin. R44/R45: MOSI and MISO pull-ups, TN-02039 table 4.3 note 4." (exclude_from_sim no) (at 330.2 127 0) (effects (font (size 1.27 1.27)) (justify left top)))
   (sheet_instances (path "/" (page "4")))
   (symbol (lib_id "device:Header_2PIN") (at 144.78 127 0) (unit 1)

Commit message: more fixes, and r2 gerber first pass
Parts:
- added R48: 100R, Resistor_SMD:R_0603_1608Metric, symbol device:R
- C37: MPN (none) -> Samsung CL10B105KA8NNNC
- C5, C6: MPN (none) -> Samsung CL10B104KO8NNNC
- R16, R17, R18, R19, R20, R21, R22, R23, R24: MPN (none) -> Yageo RC0603FR-074K7L
- R25: MPN (none) -> Yageo RC0603FR-071KL
- R26: MPN (none) -> Yageo RC0603FR-0722RL
- R27, R28, R44, R45: MPN (none) -> Yageo RC0603FR-0710KL
- R43: MPN (none) -> Yageo RC0603FR-07100RL
- SW1: MPN (none) -> Same Sky TS18-5-15-SL-260-SMT-TR
- U1: MPN (none) -> Lattice LFE5U-12F-6TG144C
- U4: MPN (none) -> Winbond W25Q128JVSIQ
- X1: MPN (none) -> ECS ECS-2520MV-250-BN-TR
Connections:
- net PROGRAMN: now also R48.1
- new net FPGA_REBOOT: R48.2
Other:
- note added: "R48: the FPGA reboots itself by pulling PROGRAMN low from pin 67 (FPGA_REBOOT), for example after rewriting the flash from the SD card. C37 and R20 bring PROGRAMN back up about 5 ms later."

Commit message: cleaning up: adding BoM for builds, part numbers, DNP flags, etc.
Parts:
- C37: LCSC (none) -> C29936
- C5, C6: LCSC (none) -> C66501
- J4: LCSC (none) -> C37208
- J6, J7: now not fitted
- R16, R17, R18, R19, R20, R21, R22, R23, R24: LCSC (none) -> C99782
- R25: LCSC (none) -> C22548
- R26: LCSC (none) -> C107701
- R27, R28, R44, R45: LCSC (none) -> C98220
- R43, R48: LCSC (none) -> C105588
- SW1: LCSC (none) -> C7074292; now not fitted
- U1: LCSC (none) -> C19979181
- U4: LCSC (none) -> C97521
- X1: LCSC (none) -> C405463
Changed lines of the file:
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@@
     (property "Description" "ECP5, built as a 25F" (at 203.2 114.3 0) (effects (font (size 1.27 1.27)) hide))
     (property "MPN" "Lattice LFE5U-12F-6TG144C" (at 203.2 114.3 0) (effects (font (size 1.27 1.27)) hide))
+    (property "LCSC" "C19979181" (at 203.2 114.3 0) (effects (font (size 1.27 1.27)) hide))
     (pin "64")
     (pin "63")
@@
     (property "Description" "resistor" (at 160.02 104.14 0) (effects (font (size 1.27 1.27)) hide))
     (property "MPN" "Yageo RC0603FR-074K7L" (at 160.02 104.14 0) (effects (font (size 1.27 1.27)) hide))
+    (property "LCSC" "C99782" (at 160.02 104.14 0) (effects (font (size 1.27 1.27)) hide))
     (pin "1")
     (pin "2")
@@
     (property "Description" "resistor" (at 152.4 104.14 0) (effects (font (size 1.27 1.27)) hide))
     (property "MPN" "Yageo RC0603FR-074K7L" (at 152.4 104.14 0) (effects (font (size 1.27 1.27)) hide))
+    (property "LCSC" "C99782" (at 152.4 104.14 0) (effects (font (size 1.27 1.27)) hide))
     (pin "1")
     (pin "2")
@@
     (property "Description" "resistor" (at 144.78 104.14 0) (effects (font (size 1.27 1.27)) hide))
     (property "MPN" "Yageo RC0603FR-074K7L" (at 144.78 104.14 0) (effects (font (size 1.27 1.27)) hide))
+    (property "LCSC" "C99782" (at 144.78 104.14 0) (effects (font (size 1.27 1.27)) hide))
     (pin "1")
     (pin "2")
@@
     (property "Description" "resistor" (at 137.16 104.14 0) (effects (font (size 1.27 1.27)) hide))
     (property "MPN" "Yageo RC0603FR-074K7L" (at 137.16 104.14 0) (effects (font (size 1.27 1.27)) hide))
+    (property "LCSC" "C99782" (at 137.16 104.14 0) (effects (font (size 1.27 1.27)) hide))
     (pin "1")
     (pin "2")
@@
   )
   (symbol (lib_id "device:SW_Push") (at 129.54 118.11 180) (unit 1)
-    (exclude_from_sim no) (in_bom yes) (on_board yes) (dnp no)
+    (exclude_from_sim no) (in_bom yes) (on_board yes) (dnp yes)
     (property "Reference" "SW1" (at 127 116.21 0) (effects (font (size 1.27 1.27)) (justify right)))
     (property "Value" "PROGRAMN button" (at 133.35 122.05 0) (effects (font (size 1.27 1.27)) (justify right) hide))
@@
     (property "Description" "tactile switch" (at 129.54 118.11 0) (effects (font (size 1.27 1.27)) hide))
     (property "MPN" "Same Sky TS18-5-15-SL-260-SMT-TR" (at 129.54 118.11 0) (effects (font (size 1.27 1.27)) hide))
+    (property "LCSC" "C7074292" (at 129.54 118.11 0) (effects (font (size 1.27 1.27)) hide))
     (pin "1")
     (pin "2")
@@
     (property "Description" "resistor" (at 228.6 107.95 0) (effects (font (size 1.27 1.27)) hide))
     (property "MPN" "Yageo RC0603FR-0722RL" (at 228.6 107.95 0) (effects (font (size 1.27 1.27)) hide))
+    (property "LCSC" "C107701" (at 228.6 107.95 0) (effects (font (size 1.27 1.27)) hide))
     (pin "1")
     (pin "2")
@@
     (property "Datasheet" "" (at 99.06 88.9 0) (effects (font (size 1.27 1.27)) hide))
     (property "Description" "JTAG, 1x6 0.1 in" (at 99.06 88.9 0) (effects (font (size 1.27 1.27)) hide))
+    (property "LCSC" "C37208" (at 99.06 88.9 0) (effects (font (size 1.27 1.27)) hide))
     (pin "1")
     (pin "2")
@@
     (property "Description" "resistor" (at 68.58 78.74 0) (effects (font (size 1.27 1.27)) hide))
     (property "MPN" "Yageo RC0603FR-074K7L" (at 68.58 78.74 0) (effects (font (size 1.27 1.27)) hide))
+    (property "LCSC" "C99782" (at 68.58 78.74 0) (effects (font (size 1.27 1.27)) hide))
     (pin "1")
     (pin "2")
@@
     (property "Description" "resistor" (at 60.96 78.74 0) (effects (font (size 1.27 1.27)) hide))
     (property "MPN" "Yageo RC0603FR-074K7L" (at 60.96 78.74 0) (effects (font (size 1.27 1.27)) hide))
+    (property "LCSC" "C99782" (at 60.96 78.74 0) (effects (font (size 1.27 1.27)) hide))
     (pin "1")
     (pin "2")
@@
     (property "Description" "resistor" (at 53.34 78.74 0) (effects (font (size 1.27 1.27)) hide))
     (property "MPN" "Yageo RC0603FR-074K7L" (at 53.34 78.74 0) (effects (font (size 1.27 1.27)) hide))
+    (property "LCSC" "C99782" (at 53.34 78.74 0) (effects (font (size 1.27 1.27)) hide))
     (pin "1")
     (pin "2")
@@
     (property "Description" "resistor" (at 68.58 99.06 0) (effects (font (size 1.27 1.27)) hide))
     (property "MPN" "Yageo RC0603FR-074K7L" (at 68.58 99.06 0) (effects (font (size 1.27 1.27)) hide))
+    (property "LCSC" "C99782" (at 68.58 99.06 0) (effects (font (size 1.27 1.27)) hide))
     (pin "1")
     (pin "2")
@@
     (property "Description" "128 Mbit SPI NOR configuration flash" (at 317.5 96.52 0) (effects (font (size 1.27 1.27)) hide))
     (property "MPN" "Winbond W25Q128JVSIQ" (at 317.5 96.52 0) (effects (font (size 1.27 1.27)) hide))
+    (property "LCSC" "C97521" (at 317.5 96.52 0) (effects (font (size 1.27 1.27)) hide))
     (pin "1")
     (pin "6")
@@
     (property "Description" "resistor" (at 288.29 83.82 0) (effects (font (size 1.27 1.27)) hide))
     (property "MPN" "Yageo RC0603FR-074K7L" (at 288.29 83.82 0) (effects (font (size 1.27 1.27)) hide))
+    (property "LCSC" "C99782" (at 288.29 83.82 0) (effects (font (size 1.27 1.27)) hide))
     (pin "1")
     (pin "2")
@@
     (property "Description" "resistor" (at 280.67 83.82 0) (effects (font (size 1.27 1.27)) hide))
     (property "MPN" "Yageo RC0603FR-071KL" (at 280.67 83.82 0) (effects (font (size 1.27 1.27)) hide))
+    (property "LCSC" "C22548" (at 280.67 83.82 0) (effects (font (size 1.27 1.27)) hide))
     (pin "1")
     (pin "2")
@@
     (property "Description" "resistor" (at 273.05 83.82 0) (effects (font (size 1.27 1.27)) hide))
     (property "MPN" "Yageo RC0603FR-0710KL" (at 273.05 83.82 0) (effects (font (size 1.27 1.27)) hide))
+    (property "LCSC" "C98220" (at 273.05 83.82 0) (effects (font (size 1.27 1.27)) hide))
     (pin "1")
     (pin "2")
@@
     (property "Description" "resistor" (at 265.43 83.82 0) (effects (font (size 1.27 1.27)) hide))
     (property "MPN" "Yageo RC0603FR-0710KL" (at 265.43 83.82 0) (effects (font (size 1.27 1.27)) hide))
+    (property "LCSC" "C98220" (at 265.43 83.82 0) (effects (font (size 1.27 1.27)) hide))
     (pin "1")
     (pin "2")
@@
     (property "Description" "capacitor" (at 297.18 81.28 0) (effects (font (size 1.27 1.27)) hide))
     (property "MPN" "Samsung CL10B104KO8NNNC" (at 297.18 81.28 0) (effects (font (size 1.27 1.27)) hide))
+    (property "LCSC" "C66501" (at 297.18 81.28 0) (effects (font (size 1.27 1.27)) hide))
     (pin "1")
     (pin "2")
@@
   )
   (symbol (lib_id "device:Header_FLASH") (at 381 96.52 0) (unit 1)
-    (exclude_from_sim no) (in_bom yes) (on_board yes) (dnp no)
+    (exclude_from_sim no) (in_bom yes) (on_board yes) (dnp yes)
     (property "Reference" "J6" (at 375.92 80.64 0) (effects (font (size 1.27 1.27)) (justify left)))
     (property "Value" "flash service 1x7" (at 375.92 83.19 0) (effects (font (size 1.27 1.27)) (justify left)))
@@
     (property "Description" "25 MHz CMOS oscillator" (at 304.8 180.34 0) (effects (font (size 1.27 1.27)) hide))
     (property "MPN" "ECS ECS-2520MV-250-BN-TR" (at 304.8 180.34 0) (effects (font (size 1.27 1.27)) hide))
+    (property "LCSC" "C405463" (at 304.8 180.34 0) (effects (font (size 1.27 1.27)) hide))
     (pin "1")
     (pin "3")
@@
     (property "Description" "capacitor" (at 284.48 171.45 0) (effects (font (size 1.27 1.27)) hide))
     (property "MPN" "Samsung CL10B104KO8NNNC" (at 284.48 171.45 0) (effects (font (size 1.27 1.27)) hide))
+    (property "LCSC" "C66501" (at 284.48 171.45 0) (effects (font (size 1.27 1.27)) hide))
     (pin "1")
     (pin "2")
@@
     (property "Description" "resistor" (at 347.98 93.98 0) (effects (font (size 1.27 1.27)) hide))
     (property "MPN" "Yageo RC0603FR-07100RL" (at 347.98 93.98 0) (effects (font (size 1.27 1.27)) hide))
+    (property "LCSC" "C105588" (at 347.98 93.98 0) (effects (font (size 1.27 1.27)) hide))
     (pin "1")
     (pin "2")
@@
     (property "Description" "resistor" (at 335.28 116.84 0) (effects (font (size 1.27 1.27)) hide))
     (property "MPN" "Yageo RC0603FR-0710KL" (at 335.28 116.84 0) (effects (font (size 1.27 1.27)) hide))
+    (property "LCSC" "C98220" (at 335.28 116.84 0) (effects (font (size 1.27 1.27)) hide))
     (pin "1")
     (pin "2")
@@
     (property "Description" "resistor" (at 342.9 116.84 0) (effects (font (size 1.27 1.27)) hide))
     (property "MPN" "Yageo RC0603FR-0710KL" (at 342.9 116.84 0) (effects (font (size 1.27 1.27)) hide))
+    (property "LCSC" "C98220" (at 342.9 116.84 0) (effects (font (size 1.27 1.27)) hide))
     (pin "1")
     (pin "2")
@@
     (property "Description" "resistor" (at 299.72 121.92 0) (effects (font (size 1.27 1.27)) hide))
     (property "MPN" "Yageo RC0603FR-07100RL" (at 299.72 121.92 0) (effects (font (size 1.27 1.27)) hide))
+    (property "LCSC" "C105588" (at 299.72 121.92 0) (effects (font (size 1.27 1.27)) hide))
     (pin "1")
     (pin "2")
@@
   (sheet_instances (path "/" (page "4")))
   (symbol (lib_id "device:Header_2PIN") (at 144.78 127 0) (unit 1)
-    (exclude_from_sim no) (in_bom yes) (on_board yes) (dnp no)
+    (exclude_from_sim no) (in_bom yes) (on_board yes) (dnp yes)
     (property "Reference" "J7" (at 142.24 121.92 0) (effects (font (size 1.27 1.27)) (justify left)))
     (property "Value" "PROGRAMN button header (optional)" (at 142.24 124.46 0) (effects (font (size 1.27 1.27)) (justify left) hide))
@@
     (property "Description" "PROGRAMN power-up delay (X7R, 10 V or more): with R20 it holds PROGRAMN low until 3V3 is above the flash's VIH, ECP5 datasheet 3.5" (at 165.1 120.65 0) (effects (font (size 1.27 1.27)) hide))
     (property "MPN" "Samsung CL10B105KA8NNNC" (at 165.1 120.65 0) (effects (font (size 1.27 1.27)) hide))
-    (pin "1")
-    (pin "2")
+    (property "LCSC" "C29936" (at 165.1 120.65 0) (effects (font (size 1.27 1.27)) hide))
+    (pin "1")
+    (pin "2")

Commit message: tuning placement and parts lists
Parts:
- J4: now not fitted
Changed lines of the file:
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@@
   (text "JTAG" (exclude_from_sim no) (at 16.51 47.5 0) (effects (font (size 2 2) bold) (justify left top)))
   (symbol (lib_id "device:Header_JTAG") (at 99.06 88.9 0) (unit 1)
-    (exclude_from_sim no) (in_bom yes) (on_board yes) (dnp no)
+    (exclude_from_sim no) (in_bom yes) (on_board yes) (dnp yes)
     (property "Reference" "J4" (at 93.98 74.3 0) (effects (font (size 1.27 1.27)) (justify left)))
     (property "Value" "JTAG 1x6" (at 93.98 76.84 0) (effects (font (size 1.27 1.27)) (justify left)))
